Commit message: fix: tcp link

File: urdf/ee/openarm_hand_arguments.xacro (robot description, xacro)
@@ -8,5 +8,5 @@
   <xacro:arg name="rpy_ee" default= "0 0 0" />
   <!-- Position offset between ee frame and tcp frame -->
-  <xacro:arg name="tcp_xyz" default="0 0.0 0.0" />
+  <xacro:arg name="tcp_xyz" default="0 -0.02 0.15" />
   <!-- Rotation offset between ee frame and tcp frame -->
   <xacro:arg name="tcp_rpy" default="0 0 0" />

File: urdf/ee/openarm_hand_macro.xacro (robot description, xacro)
@@ -2,17 +2,22 @@
 <robot xmlns:xacro="http://www.ros.org/wiki/xacro">
   <xacro:macro name="ee-inertials" params="name ee_inertials:=^">
-      <xacro:unless value="${name in ee_inertials}">${xacro.warning('No inertia properties defined for: ' + name)}</xacro:unless>
-      <xacro:if value="${name in ee_inertials}">
-        <!-- Access inertia properties of link 'name' -->
-        <xacro:property name="link_inertials" value="${ee_inertials[name]}" lazy_eval="false" />
-        <inertial>
-          <origin rpy="${link_inertials.origin.rpy}" xyz="${link_inertials.origin.xyz}" />
-          <mass value="${link_inertials.mass}" />
-          <xacro:if value="${'inertia' in link_inertials}">
-            <xacro:property name="I" value="${link_inertials.inertia}" />
-            <inertia ixx="${I.xx}" ixy="${I.xy}" ixz="${I.xz}" iyy="${I.yy}" iyz="${I.yz}" izz="${I.zz}" />
-          </xacro:if>
-        </inertial>
-      </xacro:if>
+    <xacro:unless value="${name in ee_inertials}">
+      ${xacro.warning('No inertia properties defined for: ' + name)}
+    </xacro:unless>
+    <xacro:if value="${name in ee_inertials}">
+      <xacro:property name="link_inertials" value="${ee_inertials[name]}" lazy_eval="false" />
+      <!-- Extract origin -->
+      <xacro:property name="xyz" value="${link_inertials.origin.x} ${link_inertials.origin.y} ${link_inertials.origin.z}" />
+      <xacro:property name="rpy" value="${link_inertials.origin.roll} ${link_inertials.origin.pitch} ${link_inertials.origin.yaw}" />
+      <inertial>
+        <origin xyz="${xyz}" rpy="${rpy}" />
+        <mass value="${link_inertials.mass}" />
+        <xacro:if value="${'inertia' in link_inertials}">
+          <xacro:property name="I" value="${link_inertials.inertia}" />
+          <inertia ixx="${I.xx}" ixy="${I.xy}" ixz="${I.xz}"
+                   iyy="${I.yy}" iyz="${I.yz}" izz="${I.zz}" />
+        </xacro:if>
+      </inertial>
+    </xacro:if>
   </xacro:macro>
   <xacro:macro name="ee_link_with_sc" params="name prefix rpy:='0 0 0' ee_kinematics_link">
