Commit message: Fix end effector prefixes

File: urdf/ee/ee_with_one_link.xacro (robot description, xacro)
@@ -5,5 +5,5 @@
     <xacro:property name="ee_prefix" default="robot_"/>
     <xacro:unless value="${arm_type == ''}">
-      <xacro:property name="ee_prefix" value="${arm_prefix}${arm_type}_" />
+      <xacro:property name="ee_prefix" value="openarm_${arm_prefix}" />
     </xacro:unless>
     <xacro:unless value="${connected_to == ''}">

File: urdf/ros2_control/openarm.ros2_control.xacro (robot description, xacro)
@@ -62,5 +62,5 @@
       <joint name="openarm_${arm_prefix}joint8" />
       <xacro:if value="${hand}">
-        <xacro:configure_joint joint_name="${arm_type}_finger_joint1" initial_position="0.0" />
+        <xacro:configure_joint joint_name="openarm_${arm_prefix}finger_joint1" initial_position="0.0" />
       </xacro:if>
     </ros2_control>
