Commit message: add: hand link

File: urdf/ee/openarm_hand.xacro (robot description, xacro)
@@ -58,5 +58,5 @@
       <parent link="${ee_prefix}hand" />
       <child link="${ee_prefix}right_finger" />
-      <origin xyz="0 -0.026 0.115" rpy="0 0 0" />
+      <origin xyz="0 0.00 0.015" rpy="0 0 0" />
       <axis xyz="0 -1 0" />
       <limit effort="10" lower="0.0" upper="0.044" velocity="1.0" />
@@ -65,5 +65,5 @@
       <parent link="${ee_prefix}hand" />
       <child link="${ee_prefix}left_finger" />
-      <origin xyz="0 -0.016 0.115" rpy="0 0 0" />
+      <origin xyz="0 0.012 0.015" rpy="0 0 0" />
       <axis xyz="0 1 0" />
       <limit effort="10" lower="0.0" upper="0.044" velocity="1.0" />

File: urdf/ee/openarm_hand_arguments.xacro (robot description, xacro)
@@ -4,9 +4,9 @@
   <xacro:arg name="special_connection" default="" />
   <!-- Position offset between ee and parent frame -->
-  <xacro:arg name="xyz_ee" default="0 0 0.0" />
+  <xacro:arg name="xyz_ee" default="0 -0.025 0.1001" />
   <!-- Rotation offset between ee and parent frame -->
   <xacro:arg name="rpy_ee" default= "0 0 0" />
   <!-- Position offset between ee frame and tcp frame -->
-  <xacro:arg name="tcp_xyz" default="0 -0.02 0.15" />
+  <xacro:arg name="tcp_xyz" default="0 -0.0 0.08" />
   <!-- Rotation offset between ee frame and tcp frame -->
   <xacro:arg name="tcp_rpy" default="0 0 0" />

File: urdf/ee/openarm_hand_macro.xacro (robot description, xacro)
@@ -7,5 +7,4 @@
     <xacro:if value="${name in ee_inertials}">
       <xacro:property name="link_inertials" value="${ee_inertials[name]}" lazy_eval="false" />
-      <!-- Extract origin -->
       <xacro:property name="xyz" value="${link_inertials.origin.x} ${link_inertials.origin.y} ${link_inertials.origin.z}" />
       <xacro:property name="rpy" value="${link_inertials.origin.roll} ${link_inertials.origin.pitch} ${link_inertials.origin.yaw}" />

Commit message: fix: physical parameter

File: urdf/ee/openarm_hand.xacro (robot description, xacro)
@@ -60,5 +60,5 @@
       <origin xyz="0 0.00 0.015" rpy="0 0 0" />
       <axis xyz="0 -1 0" />
-      <limit effort="10" lower="0.0" upper="0.044" velocity="1.0" />
+      <limit effort="333" lower="0.0" upper="0.044" velocity="10.0" />
     </joint>
     <joint name="${ee_prefix}finger_joint2" type="prismatic">
@@ -67,5 +67,5 @@
       <origin xyz="0 0.012 0.015" rpy="0 0 0" />
       <axis xyz="0 1 0" />
-      <limit effort="10" lower="0.0" upper="0.044" velocity="1.0" />
+      <limit effort="333" lower="0.0" upper="0.044" velocity="10.0" />
       <mimic joint="${ee_prefix}finger_joint1" />
     </joint>
