Commit message: repair dir structure

File: urdf/ee/openarm_hand_macro.xacro (robot description, xacro)
@@ -25,5 +25,5 @@
         <xacro:openarm-ee-kinematics-link config="${ee_kinematics_link}" name="${name}" />
         <geometry>
-          <mesh filename="package://${description_pkg}/meshes/ee/${ee_type}/visual/${name}.dae" scale="0.001 0.001 0.001" />
+          <mesh filename="package://${description_pkg}/meshes/ee/${ee_type}/visual/${name}.stl" scale="0.001 0.001 0.001" />
         </geometry>
       </visual>

File: urdf/robot/openarm_robot.xacro (robot description, xacro)
@@ -14,4 +14,5 @@
             body_kinematics_link
             ee_kinematics_link
+            ee_inertials
             parent:='world'
             xyz:='0 0 0'
@@ -44,11 +45,8 @@
     <xacro:include filename="$(find openarm_description)/urdf/body/openarm_body_macro.xacro" />
     <xacro:include filename="$(find openarm_description)/urdf/body/openarm_body.xacro" />
-    <xacro:include filename="$(find openarm_description)/urdf/ee/openarm_hand.xacro" />
+    <xacro:include filename="$(find openarm_description)/urdf/ee/ee_dispatcher.xacro" />
     <xacro:include filename="$(find openarm_description)/urdf/ee/openarm_hand_macro.xacro" />
     <xacro:include filename="$(find openarm_description)/urdf/ros2_control/openarm.ros2_control.xacro" />
     <xacro:include filename="$(find openarm_description)/urdf/ros2_control/openarm.bimanual.ros2_control.xacro" />
-    <xacro:if value="${ee_type != 'none'}">
-        <xacro:include filename="$(find openarm_description)/urdf/ee/${ee_type}_arguments.xacro" />
-    </xacro:if>
     <xacro:property name="arm_prefix_modified" value="${'' if arm_prefix == '' else arm_prefix + '_'}" />
     <xacro:property name="body_prefix_modified" value="${'' if body_prefix == '' else body_prefix + '_'}" />
@@ -106,32 +104,22 @@
             hand="${hand}"/>
         </xacro:if>
-        <xacro:if value="$(eval hand and ee_type == 'openarm_hand')">
-            <xacro:openarm_hand
+        <xacro:if value="${hand}">
+            <xacro:openarm_ee
                 connected_to="openarm_left_link7"
                 arm_type="${arm_type}"
                 arm_prefix="left_"
                 ee_type="${ee_type}"
-                ee_kinematics_link="${xacro.load_yaml('$(find openarm_description)/config/hand/openarm_hand/kinematics_link.yaml')}"
-                ee_inertials="${xacro.load_yaml('$(find openarm_description)/config/hand/openarm_hand/inertials.yaml')}"
-                rpy_ee="$(arg rpy_ee)"
-                xyz_ee="$(arg xyz_ee)"
-                tcp_xyz="$(arg tcp_xyz)"
-                tcp_rpy="$(arg tcp_rpy)"
-                description_pkg="$(arg description_pkg)"
+                ee_kinematics_link="${ee_kinematics_link}"
+                ee_inertials="${ee_inertials}"
             />
-            <xacro:openarm_hand
+            <xacro:openarm_ee
                 connected_to="openarm_right_link7"
                 arm_type="${arm_type}"
                 arm_prefix="right_"
                 ee_type="${ee_type}"
-                ee_kinematics_link="${xacro.load_yaml('$(find openarm_description)/config/hand/openarm_hand/kinematics_link.yaml')}"
-                ee_inertials="${xacro.load_yaml('$(find openarm_description)/config/hand/openarm_hand/inertials.yaml')}"
-                rpy_ee="$(arg rpy_ee)"
-                xyz_ee="$(arg xyz_ee)"
-                tcp_xyz="$(arg tcp_xyz)"
-                tcp_rpy="$(arg tcp_rpy)"
-                description_pkg="$(arg description_pkg)"
+                ee_kinematics_link="${ee_kinematics_link}"
+                ee_inertials="${ee_inertials}"
             />
-          </xacro:if>
+        </xacro:if>
     </xacro:if>
     <xacro:if value="${not bimanual}">
@@ -160,22 +148,13 @@
             can_fd="${can_fd}"/>
         </xacro:if>
-        <xacro:if value="${hand and ee_type == 'openarm_hand'}">
-        <xacro:property name="special_connection" value="$(arg special_connection)" />
-        <!-- <xacro:property name="connection" value="${special_connection if special_connection != '' else arm_type + '_link7'}" /> -->
-        <xacro:property name="connection" value="${special_connection if special_connection != '' else 'openarm' + '_link7'}" />
-        <xacro:if value="$(eval hand and ee_type == 'openarm_hand')">
-        <xacro:openarm_hand
-            connected_to="${arm_prefix_modified}${connection}"
-            arm_type="${arm_type}"
-            arm_prefix="${arm_prefix_modified}"
-            ee_type="${ee_type}"
-            ee_kinematics_link="${xacro.load_yaml('$(find openarm_description)/config/hand/openarm_hand/kinematics_link.yaml')}"
-            ee_inertials="${xacro.load_yaml('$(find openarm_description)/config/hand/openarm_hand/inertials.yaml')}"
-            rpy_ee="$(arg rpy_ee)"
-            xyz_ee="$(arg xyz_ee)"
-            tcp_xyz="$(arg tcp_xyz)"
-            tcp_rpy="$(arg tcp_rpy)"
-            description_pkg="$(arg description_pkg)"/>
-        </xacro:if>
+        <xacro:if value="${hand}">
+            <xacro:openarm_ee
+                connected_to="openarm_link7"
+                arm_type="${arm_type}"
+                arm_prefix="${arm_prefix_modified}"
+                ee_type="${ee_type}"
+                ee_kinematics_link="${ee_kinematics_link}"
+                ee_inertials="${ee_inertials}"
+            />
         </xacro:if>
         </xacro:if>

File: urdf/robot/v10/v10.urdf.xacro (robot description, xacro)
@@ -4,5 +4,5 @@
   <xacro:arg name="arm_type" default="v10" />
   <xacro:arg name="body_type" default="v10" />
-  <xacro:arg name="ee_type" default="openarm_hand" />
+  <xacro:arg name="ee_type" default="parallel_gripper" />
   <xacro:arg name="no_prefix" default="false"/>
   <xacro:arg name="hand" default="true" />
@@ -39,5 +39,6 @@
   body_kinematics="${xacro.load_yaml('$(find openarm_description)/config/body/v10/kinematics.yaml')}"
   body_kinematics_link="${xacro.load_yaml('$(find openarm_description)/config/body/v10/kinematics.yaml')}"
-  ee_kinematics_link="${xacro.load_yaml('$(find openarm_description)/config/hand/openarm_hand/kinematics_link.yaml')}"
+  ee_kinematics_link="${xacro.load_yaml('$(find openarm_description)/config/hand/parallel_link/kinematics_link.yaml')}"
+  ee_inertials="${xacro.load_yaml('$(find openarm_description)/config/hand/parallel_link/inertials.yaml')}"
   hand="$(arg hand)"
   ee_type="$(arg ee_type)"

File: urdf/robot/v20/v20.urdf.xacro (robot description, xacro)
@@ -4,5 +4,5 @@
   <xacro:arg name="arm_type" default="v20" />
   <xacro:arg name="body_type" default="v20" />
-  <xacro:arg name="ee_type" default="openarm_v20_hand" />
+  <xacro:arg name="ee_type" default="pinch_gripper" />
   <xacro:arg name="no_prefix" default="false"/>
   <xacro:arg name="hand" default="true" />
@@ -39,5 +39,6 @@
   body_kinematics="${xacro.load_yaml('$(find openarm_description)/config/body/v20/kinematics.yaml')}"
   body_kinematics_link="${xacro.load_yaml('$(find openarm_description)/config/body/v20/kinematics_link.yaml')}"
-  ee_kinematics_link="${xacro.load_yaml('$(find openarm_description)/config/hand/openarm_hand/kinematics_link.yaml')}"
+  ee_kinematics_link="${xacro.load_yaml('$(find openarm_description)/config/hand/pinch_gripper/kinematics_link.yaml')}"
+  ee_inertials="${xacro.load_yaml('$(find openarm_description)/config/hand/pinch_gripper/inertials.yaml')}"
   hand="$(arg hand)"
   ee_type="$(arg ee_type)"

Commit message: add temp finger

File: urdf/ee/openarm_hand_macro.xacro (robot description, xacro)
@@ -20,10 +20,10 @@
     </xacro:if>
   </xacro:macro>
-  <xacro:macro name="ee_link_with_sc" params="name prefix rpy:='0 0 0' ee_kinematics_link">
+  <xacro:macro name="ee_link_with_sc" params="name prefix rpy:='0 0 0' ee_kinematics_link reflect:=1">
     <link name="${prefix}${name}">
       <visual name="${prefix}${name}_visual">
         <xacro:openarm-ee-kinematics-link config="${ee_kinematics_link}" name="${name}" />
         <geometry>
-          <mesh filename="package://${description_pkg}/meshes/ee/${ee_type}/visual/${name}.stl" scale="0.001 0.001 0.001" />
+          <mesh filename="package://${description_pkg}/meshes/ee/${ee_type}/visual/${name}.dae" scale="0.001 ${0.001*reflect} 0.001" />
         </geometry>
       </visual>
@@ -31,10 +31,10 @@
         <xacro:openarm-ee-kinematics-link config="${ee_kinematics_link}" name="${name}" />
         <geometry>
-          <mesh filename="package://openarm_description/meshes/ee/${ee_type}/collision/${name}.stl" scale="0.001 0.001 0.001" />
+          <mesh filename="package://openarm_description/meshes/ee/${ee_type}/collision/${name}.stl" scale="0.001 ${0.001*reflect} 0.001" />
         </geometry>
       </collision>
       <xacro:ee-inertials name="${name}" />
     </link>
-  </xacro:macro>
+</xacro:macro>
   <xacro:macro name="openarm-ee-kinematics" params="config name">
       <xacro:property name="kinematics" value="${config[name]['kinematic']}" lazy_eval="false" />
@@ -47,3 +47,22 @@
             xyz="${kinematics_link.x} ${kinematics_link.y} ${kinematics_link.z}" />
   </xacro:macro>
+  <xacro:macro name="ee_finger_link_with_sc" params="name prefix ee_kinematics_link arm_reflect:=1 finger_reflect:=1">
+    <link name="${prefix}${name}">
+      <visual name="${prefix}${name}_visual">
+        <xacro:openarm-ee-kinematics-link config="${ee_kinematics_link}" name="${name}" />
+        <geometry>
+          <mesh filename="package://${description_pkg}/meshes/ee/${ee_type}/visual/finger.dae"
+                scale="${0.001*finger_reflect} ${0.001*arm_reflect} 0.001" />
+        </geometry>
+      </visual>
+      <collision name="${prefix}${name}_collision">
+        <xacro:openarm-ee-kinematics-link config="${ee_kinematics_link}" name="${name}" />
+        <geometry>
+          <mesh filename="package://openarm_description/meshes/ee/${ee_type}/collision/finger.stl"
+                scale="${0.001*finger_reflect} ${0.001*arm_reflect} 0.001" />
+        </geometry>
+      </collision>
+      <xacro:ee-inertials name="${name}" />
+    </link>
+</xacro:macro>
 </robot>

File: urdf/ee/pinch_gripper/openarm_v20_hand.xacro (robot description, xacro)
@@ -1,15 +1,14 @@
 <?xml version="1.0" encoding="utf-8"?>
 <robot xmlns:xacro="http://www.ros.org/wiki/xacro" name="hand">
-  <!-- safety_distance: Minimum safety distance in [m] by which the collision volumes are expanded and which is enforced during robot motions -->
   <xacro:macro name="openarm_v20_hand" params="connected_to:='' arm_type arm_prefix:='' ee_type ee_inertials ee_kinematics_link rpy_ee:='0 0 0' xyz_ee:='0 0 0' tcp_xyz:='0 0 0' tcp_rpy:='0 0 0' description_pkg:=openarm_description">
-    <xacro:property name="ee_prefix" default=""/>
+    <xacro:property name="ee_prefix" value=""/>
     <xacro:unless value="${arm_type == ''}">
-      <!-- <xacro:property name="ee_prefix" value="${arm_prefix}${arm_type}_" /> -->
       <xacro:property name="ee_prefix" value="openarm_${arm_prefix}" />
     </xacro:unless>
-    <xacro:ee_link_with_sc name="hand" prefix="${ee_prefix}" ee_kinematics_link="${ee_kinematics_link}"/>
-    <!-- <link name="${ee_prefix}hand"/> -->
+    <xacro:property name="reflect" value="${-1 if arm_prefix == 'left_' else 1}" />
+    <!-- hand link -->
+    <xacro:ee_link_with_sc name="hand" prefix="${ee_prefix}" ee_kinematics_link="${ee_kinematics_link}" reflect="${reflect}"/>
+    <!-- hand joint -->
     <xacro:unless value="${connected_to == ''}">
-      <!-- <joint name="${ee_prefix}hand_joint" type="fixed"> -->
       <joint name="${arm_prefix}openarm_hand_joint" type="fixed">
         <parent link="${connected_to}" />
@@ -18,5 +17,5 @@
       </joint>
     </xacro:unless>
-    <!-- Define the hand_tcp frame -->
+    <!-- tcp frame -->
     <link name="${ee_prefix}hand_tcp" />
     <joint name="${ee_prefix}hand_tcp_joint" type="fixed">
@@ -25,48 +24,34 @@
       <child link="${ee_prefix}hand_tcp" />
     </joint>
-    <link name="${ee_prefix}left_finger">
-      <visual name="${ee_prefix}left_finger_visual">
-        <xacro:openarm-ee-kinematics-link config="${ee_kinematics_link}" name="left_finger" />
-        <geometry>
-          <mesh filename="package://${description_pkg}/meshes/ee/${ee_type}/visual/finger_left.stl" scale="0.001 0.001 0.001"/>
-        </geometry>
-      </visual>
-      <collision name="${ee_prefix}left_finger_collision">
-        <xacro:openarm-ee-kinematics-link config="${ee_kinematics_link}" name="left_finger" />
-        <geometry>
-          <mesh filename="package://${description_pkg}/meshes/ee/${ee_type}/collision/finger.stl" scale="0.001 0.001 0.001" />
-        </geometry>
-      </collision>
-      <xacro:ee-inertials name="left_finger"/>
-    </link>
-    <link name="${ee_prefix}right_finger">
-      <visual name="${ee_prefix}right_finger_visual">
-        <xacro:openarm-ee-kinematics-link config="${ee_kinematics_link}" name="right_finger" />
-        <geometry>
-          <mesh filename="package://${description_pkg}/meshes/ee/${ee_type}/visual/finger_left.stl" scale="0.001 -0.001 0.001"/>
-        </geometry>
-      </visual>
-      <collision name="${ee_prefix}right_finger_collision">
-        <xacro:openarm-ee-kinematics-link config="${ee_kinematics_link}" name="right_finger" />
-        <geometry>
-          <mesh filename="package://${description_pkg}/meshes/ee/${ee_type}/collision/finger.stl" scale="0.001 -0.001 0.001" />
-        </geometry>
-      </collision>
-      <xacro:ee-inertials name="right_finger"/>
-    </link>
+    <!-- finger links -->
+    <xacro:ee_finger_link_with_sc
+        name="right_finger"
+        prefix="${ee_prefix}"
+        ee_kinematics_link="${ee_kinematics_link}"
+        arm_reflect="${reflect}"
+        finger_reflect="-1"
+    />
+    <xacro:ee_finger_link_with_sc
+        name="left_finger"
+        prefix="${ee_prefix}"
+        ee_kinematics_link="${ee_kinematics_link}"
+        arm_reflect="${reflect}"
+        finger_reflect="1"
+    />
+    <!-- finger joints -->
     <joint name="${ee_prefix}finger_joint1" type="revolute">
-        <parent link="${ee_prefix}hand" />
-        <child link="${ee_prefix}right_finger" />
-        <origin xyz="0 -0.006 0.015" rpy="0 0 0" />
-        <axis xyz="1 0 0" />
-        <limit effort="333" lower="0.0" upper="1.5708" velocity="10.0" />
+      <parent link="${ee_prefix}hand" />
+      <child link="${ee_prefix}right_finger" />
+      <origin xyz="0 0.006 0.015" rpy="0 0 0" />
+      <axis xyz="0 1 0" />
+      <limit effort="333" lower="0.0" upper="1.5708" velocity="10.0" />
     </joint>
     <joint name="${ee_prefix}finger_joint2" type="revolute">
-        <parent link="${ee_prefix}hand" />
-        <child link="${ee_prefix}left_finger" />
-        <origin xyz="0 0.006 0.015" rpy="0 0 0" />
-        <axis xyz="-1 0 0" />
-        <limit effort="333" lower="0.0" upper="1.5708" velocity="10.0" />
-        <mimic joint="${ee_prefix}finger_joint1" />
+      <parent link="${ee_prefix}hand" />
+      <child link="${ee_prefix}left_finger" />
+      <origin xyz="0 -0.006 0.015" rpy="0 0 0" />
+      <axis xyz="0 -1 0" />
+      <limit effort="333" lower="0.0" upper="1.5708" velocity="10.0" />
+      <mimic joint="${ee_prefix}finger_joint1" />
     </joint>
   </xacro:macro>
