Commit message: add finger kin yaml

File: urdf/ee/ee_dispatcher.xacro (robot description, xacro)
@@ -3,5 +3,5 @@
   <xacro:include filename="$(find openarm_description)/urdf/ee/parallel_link/openarm_parallel_gripper.xacro" />
   <xacro:include filename="$(find openarm_description)/urdf/ee/pinch_gripper/openarm_v20_pinch_gripper.xacro" />
-  <xacro:macro name="openarm_ee" params="ee_type connected_to arm_type arm_prefix ee_kinematics_link ee_inertials">
+  <xacro:macro name="openarm_ee" params="ee_type connected_to arm_type arm_prefix ee_kinematics ee_kinematics_link ee_inertials">
     <xacro:if value="${ee_type == 'parallel_link'}">
       <xacro:openarm_parallel_gripper
@@ -10,4 +10,5 @@
         arm_prefix="${arm_prefix}"
         ee_type="${ee_type}"
+        ee_kinematics="${ee_kinematics}"
         ee_kinematics_link="${ee_kinematics_link}"
         ee_inertials="${ee_inertials}"
@@ -20,4 +21,5 @@
         arm_prefix="${arm_prefix}"
         ee_type="${ee_type}"
+        ee_kinematics="${ee_kinematics}"
         ee_kinematics_link="${ee_kinematics_link}"
         ee_inertials="${ee_inertials}"

File: urdf/ee/parallel_link/openarm_parallel_gripper.xacro (robot description, xacro)
@@ -1,5 +1,5 @@
 <?xml version="1.0" encoding="utf-8"?>
 <robot xmlns:xacro="http://www.ros.org/wiki/xacro" name="parallel_gripper">
-  <xacro:macro name="openarm_parallel_gripper" params="connected_to:='' arm_type arm_prefix:='' ee_type ee_inertials ee_kinematics_link rpy_ee:='0 0 0' xyz_ee:='0 0 0' tcp_xyz:='0 0 0' tcp_rpy:='0 0 0' description_pkg:=openarm_description">
+  <xacro:macro name="openarm_parallel_gripper" params="connected_to:='' arm_type arm_prefix:='' ee_type ee_inertials ee_kinematics ee_kinematics_link rpy_ee:='0 0 0' xyz_ee:='0 0 0' tcp_xyz:='0 0 0' tcp_rpy:='0 0 0' description_pkg:=openarm_description">
     <xacro:property name="ee_prefix" default=""/>
     <xacro:unless value="${arm_type == ''}">
@@ -42,6 +42,22 @@
     </link>
     <joint name="${ee_prefix}finger_joint1" type="prismatic">
+        <parent link="${connected_to}" />
+        <child link="${ee_prefix}right_finger" />
+        <xacro:openarm-ee-kinematics config="${ee_kinematics}" name="finger_joint" />
+        <axis xyz="0 -1 0" />
+        <limit effort="333" lower="0.0" upper="0.044" velocity="10.0" />
+    </joint>
+    <joint name="${ee_prefix}finger_joint2" type="prismatic">
+        <parent link="${connected_to}" />
+        <child link="${ee_prefix}left_finger" />
+        <xacro:property name="fj" value="${ee_kinematics['finger_joint']['kinematic']}" />
+        <origin xyz="${fj.x} ${-fj.y} ${fj.z}" rpy="0 0 0" />
+        <axis xyz="0 1 0" />
+        <limit effort="333" lower="0.0" upper="0.044" velocity="10.0" />
+        <mimic joint="${ee_prefix}finger_joint1" />
+    </joint>
+    <!-- <joint name="${ee_prefix}finger_joint1" type="prismatic">
       <parent link="${connected_to}" /> <child link="${ee_prefix}right_finger" />
-      <origin xyz="0 -0.006 0.015" rpy="0 0 0" />
+      <origin xyz="0 -0.006 0.115" rpy="0 0 0" />
       <axis xyz="0 -1 0" />
       <limit effort="333" lower="0.0" upper="0.044" velocity="10.0" />
@@ -49,9 +65,9 @@
     <joint name="${ee_prefix}finger_joint2" type="prismatic">
       <parent link="${connected_to}" /> <child link="${ee_prefix}left_finger" />
-      <origin xyz="0 0.006 0.015" rpy="0 0 0" />
+      <origin xyz="0 0.006 0.115" rpy="0 0 0" />
       <axis xyz="0 1 0" />
       <limit effort="333" lower="0.0" upper="0.044" velocity="10.0" />
       <mimic joint="${ee_prefix}finger_joint1" />
-    </joint>
+    </joint> -->
   </xacro:macro>
 </robot>

File: urdf/ee/pinch_gripper/openarm_v20_pinch_gripper.xacro (robot description, xacro)
@@ -1,4 +1,4 @@
 <?xml version="1.0" encoding="utf-8"?>
-<robot xmlns:xacro="http://www.ros.org/wiki/xacro" name="pinch_gripper"> <xacro:macro name="openarm_v20_pinch_gripper" params="connected_to:='' arm_type arm_prefix:='' ee_type ee_inertials ee_kinematics_link rpy_ee:='0 0 0' xyz_ee:='0 0 0' tcp_xyz:='0 0 0' tcp_rpy:='0 0 0' description_pkg:=openarm_description">
+<robot xmlns:xacro="http://www.ros.org/wiki/xacro" name="pinch_gripper"> <xacro:macro name="openarm_v20_pinch_gripper" params="connected_to:='' arm_type arm_prefix:='' ee_type ee_inertials ee_kinematics ee_kinematics_link rpy_ee:='0 0 0' xyz_ee:='0 0 0' tcp_xyz:='0 0 0' tcp_rpy:='0 0 0' description_pkg:=openarm_description">
     <xacro:property name="ee_prefix" value=""/>
     <xacro:unless value="${arm_type == ''}">
@@ -25,4 +25,21 @@
         finger_reflect="1"
     />
+<joint name="${ee_prefix}finger_joint1" type="revolute">
+    <parent link="${connected_to}" />
+    <child link="${ee_prefix}right_finger" />
+    <xacro:openarm-ee-kinematics config="${ee_kinematics}" name="finger_joint" />
+    <axis xyz="0 1 0" />
+    <limit effort="333" lower="0.0" upper="1.5708" velocity="10.0" />
+</joint>
+<joint name="${ee_prefix}finger_joint2" type="revolute">
+    <parent link="${connected_to}" />
+    <child link="${ee_prefix}left_finger" />
+    <xacro:property name="fj" value="${ee_kinematics['finger_joint']['kinematic']}" />
+    <origin xyz="${fj.x} ${-fj.y} ${fj.z}" rpy="${fj.roll} ${fj.pitch} ${fj.yaw}" />
+    <axis xyz="0 -1 0" />
+    <limit effort="333" lower="0.0" upper="1.5708" velocity="10.0" />
+    <mimic joint="${ee_prefix}finger_joint1" />
+</joint>
+<!--
     <joint name="${ee_prefix}finger_joint1" type="revolute">
       <parent link="${connected_to}" /> <child link="${ee_prefix}right_finger" />
@@ -35,5 +52,5 @@
       <limit effort="333" lower="0.0" upper="1.5708" velocity="10.0" />
       <mimic joint="${ee_prefix}finger_joint1" />
-    </joint>
+    </joint> -->
   </xacro:macro>
 </robot>

File: urdf/robot/openarm_robot.xacro (robot description, xacro)
@@ -13,4 +13,5 @@
             body_kinematics
             body_kinematics_link
+            ee_kinematics
             ee_kinematics_link
             ee_inertials
@@ -95,4 +96,5 @@
             arm_prefix="left_"
             ee_type="${ee_type}"
+            ee_kinematics="${ee_kinematics}"
             ee_kinematics_link="${ee_kinematics_link}"
             ee_inertials="${ee_inertials}"
@@ -103,4 +105,5 @@
             arm_prefix="right_"
             ee_type="${ee_type}"
+            ee_kinematics="${ee_kinematics}"
             ee_kinematics_link="${ee_kinematics_link}"
             ee_inertials="${ee_inertials}"
@@ -137,4 +140,5 @@
             arm_prefix="${arm_prefix_modified}"
             ee_type="${ee_type}"
+            ee_kinematics="${ee_kinematics}"
             ee_kinematics_link="${ee_kinematics_link}"
             ee_inertials="${ee_inertials}"

File: urdf/robot/v10/v10.urdf.xacro (robot description, xacro)
@@ -33,6 +33,7 @@
   body_kinematics="${xacro.load_yaml('$(find openarm_description)/config/body/$(arg body_type)/kinematics.yaml')}"
   body_kinematics_link="${xacro.load_yaml('$(find openarm_description)/config/body/$(arg body_type)/kinematics.yaml')}"
+  ee_inertials="${xacro.load_yaml('$(find openarm_description)/config/ee/' + auto_ee_type + '/inertials.yaml')}"
+  ee_kinematics="${xacro.load_yaml('$(find openarm_description)/config/ee/' + auto_ee_type + '/kinematics.yaml')}"
   ee_kinematics_link="${xacro.load_yaml('$(find openarm_description)/config/ee/' + auto_ee_type + '/kinematics_link.yaml')}"
-  ee_inertials="${xacro.load_yaml('$(find openarm_description)/config/ee/' + auto_ee_type + '/inertials.yaml')}"
   ee_type="${auto_ee_type}" ros2_control="$(arg ros2_control)"
   can_interface="$(arg can_interface)"

File: urdf/robot/v20/v20.urdf.xacro (robot description, xacro)
@@ -35,4 +35,5 @@
   body_kinematics="${xacro.load_yaml('$(find openarm_description)/config/body/$(arg body_type)/kinematics.yaml')}"
   body_kinematics_link="${xacro.load_yaml('$(find openarm_description)/config/body/$(arg body_type)/kinematics_link.yaml')}"
+  ee_kinematics="${xacro.load_yaml('$(find openarm_description)/config/ee/' + auto_ee_type + '/kinematics.yaml')}"
   ee_kinematics_link="${xacro.load_yaml('$(find openarm_description)/config/ee/' + auto_ee_type + '/kinematics_link.yaml')}"
   ee_inertials="${xacro.load_yaml('$(find openarm_description)/config/ee/' + auto_ee_type + '/inertials.yaml')}"

Commit message: fix and pass yaml to ee

File: urdf/ee/ee_dispatcher.xacro (robot description, xacro)
@@ -3,5 +3,5 @@
   <xacro:include filename="$(find openarm_description)/urdf/ee/parallel_link/openarm_parallel_gripper.xacro" />
   <xacro:include filename="$(find openarm_description)/urdf/ee/pinch_gripper/openarm_v20_pinch_gripper.xacro" />
-  <xacro:macro name="openarm_ee" params="ee_type connected_to arm_type arm_prefix ee_kinematics ee_kinematics_link ee_inertials">
+  <xacro:macro name="openarm_ee" params="ee_type connected_to arm_type arm_prefix ee_kinematics ee_kinematics_link ee_inertials ee_joints_limits rpy_ee:='0 0 0' xyz_ee:='0 0 0' tcp_xyz:='0 0 0' tcp_rpy:='0 0 0' description_pkg:=openarm_description">
     <xacro:if value="${ee_type == 'parallel_link'}">
       <xacro:openarm_parallel_gripper
@@ -13,4 +13,5 @@
         ee_kinematics_link="${ee_kinematics_link}"
         ee_inertials="${ee_inertials}"
+        ee_joints_limits="${ee_joints_limits}"
       />
     </xacro:if>
@@ -24,4 +25,5 @@
         ee_kinematics_link="${ee_kinematics_link}"
         ee_inertials="${ee_inertials}"
+        ee_joints_limits="${ee_joints_limits}"
       />
     </xacro:if>

File: urdf/ee/parallel_link/openarm_parallel_gripper.xacro (robot description, xacro)
@@ -1,5 +1,5 @@
 <?xml version="1.0" encoding="utf-8"?>
 <robot xmlns:xacro="http://www.ros.org/wiki/xacro" name="parallel_gripper">
-  <xacro:macro name="openarm_parallel_gripper" params="connected_to:='' arm_type arm_prefix:='' ee_type ee_inertials ee_kinematics ee_kinematics_link rpy_ee:='0 0 0' xyz_ee:='0 0 0' tcp_xyz:='0 0 0' tcp_rpy:='0 0 0' description_pkg:=openarm_description">
+  <xacro:macro name="openarm_parallel_gripper" params="connected_to:='' arm_type arm_prefix:='' ee_type ee_inertials ee_kinematics ee_kinematics_link ee_joints_limits rpy_ee:='0 0 0' xyz_ee:='0 0 0' tcp_xyz:='0 0 0' tcp_rpy:='0 0 0' description_pkg:=openarm_description">
     <xacro:property name="ee_prefix" default=""/>
     <xacro:unless value="${arm_type == ''}">

File: urdf/ee/pinch_gripper/openarm_v20_pinch_gripper.xacro (robot description, xacro)
@@ -1,4 +1,4 @@
 <?xml version="1.0" encoding="utf-8"?>
-<robot xmlns:xacro="http://www.ros.org/wiki/xacro" name="pinch_gripper"> <xacro:macro name="openarm_v20_pinch_gripper" params="connected_to:='' arm_type arm_prefix:='' ee_type ee_inertials ee_kinematics ee_kinematics_link rpy_ee:='0 0 0' xyz_ee:='0 0 0' tcp_xyz:='0 0 0' tcp_rpy:='0 0 0' description_pkg:=openarm_description">
+<robot xmlns:xacro="http://www.ros.org/wiki/xacro" name="pinch_gripper"> <xacro:macro name="openarm_v20_pinch_gripper" params="connected_to:='' arm_type arm_prefix:='' ee_type ee_inertials ee_kinematics ee_kinematics_link ee_joints_limits rpy_ee:='0 0 0' xyz_ee:='0 0 0' tcp_xyz:='0 0 0' tcp_rpy:='0 0 0' description_pkg:=openarm_description">
     <xacro:property name="ee_prefix" value=""/>
     <xacro:unless value="${arm_type == ''}">
@@ -25,5 +25,27 @@
         finger_reflect="1"
     />
-<joint name="${ee_prefix}finger_joint1" type="revolute">
+  <joint name="${ee_prefix}finger_joint1" type="revolute">
+      <parent link="${connected_to}" />
+      <child link="${ee_prefix}right_finger" />
+      <xacro:openarm-ee-kinematics config="${ee_kinematics}" name="finger_joint" />
+      <axis xyz="0 1 0" />
+      <limit effort="${ee_joints_limits['finger_joint']['limit']['effort']}"
+            lower="${ee_joints_limits['finger_joint']['limit']['lower']}"
+            upper="${ee_joints_limits['finger_joint']['limit']['upper']}"
+            velocity="${ee_joints_limits['finger_joint']['limit']['velocity']}" />
+  </joint>
+  <joint name="${ee_prefix}finger_joint2" type="revolute">
+      <parent link="${connected_to}" />
+      <child link="${ee_prefix}left_finger" />
+      <xacro:property name="fj" value="${ee_kinematics['finger_joint']['kinematic']}" />
+      <origin xyz="${fj.x} ${-fj.y} ${fj.z}" rpy="${fj.roll} ${fj.pitch} ${fj.yaw}" />
+      <axis xyz="0 -1 0" />
+      <limit effort="${ee_joints_limits['finger_joint']['limit']['effort']}"
+            lower="${ee_joints_limits['finger_joint']['limit']['lower']}"
+            upper="${ee_joints_limits['finger_joint']['limit']['upper']}"
+            velocity="${ee_joints_limits['finger_joint']['limit']['velocity']}" />
+      <mimic joint="${ee_prefix}finger_joint1" />
+  </joint>
+<!-- <joint name="${ee_prefix}finger_joint1" type="revolute">
     <parent link="${connected_to}" />
     <child link="${ee_prefix}right_finger" />
@@ -40,5 +62,5 @@
     <limit effort="333" lower="0.0" upper="1.5708" velocity="10.0" />
     <mimic joint="${ee_prefix}finger_joint1" />
-</joint>
+</joint> -->
 <!--
     <joint name="${ee_prefix}finger_joint1" type="revolute">

File: urdf/robot/openarm_robot.xacro (robot description, xacro)
@@ -16,4 +16,5 @@
             ee_kinematics_link
             ee_inertials
+            ee_joints_limits
             parent:='world'
             xyz:='0 0 0'
@@ -99,4 +100,5 @@
             ee_kinematics_link="${ee_kinematics_link}"
             ee_inertials="${ee_inertials}"
+            ee_joints_limits="${ee_joints_limits}"
         />
         <xacro:openarm_ee
@@ -108,4 +110,5 @@
             ee_kinematics_link="${ee_kinematics_link}"
             ee_inertials="${ee_inertials}"
+            ee_joints_limits="${ee_joints_limits}"
         />
         <!-- ros2_control hardware interfaces for bimanual setup -->
@@ -120,5 +123,6 @@
             left_arm_prefix="${left_arm_prefix}"
             right_arm_prefix="${right_arm_prefix}"
-            hand="true"/>
+            hand="true"
+            ee_type="${ee_type}"/>
         </xacro:if>
     </xacro:if>
@@ -143,4 +147,5 @@
             ee_kinematics_link="${ee_kinematics_link}"
             ee_inertials="${ee_inertials}"
+            ee_joints_limits="${ee_joints_limits}"
         />
         <xacro:if value="${ros2_control}">
@@ -153,5 +158,7 @@
                 fake_sensor_commands="${fake_sensor_commands}"
                 hand="true"
-                can_fd="${can_fd}"/> </xacro:if>
+                can_fd="${can_fd}"
+                ee_type="${ee_type}"/>
+        </xacro:if>
     </xacro:if>
   </xacro:macro>

File: urdf/robot/v10/v10.urdf.xacro (robot description, xacro)
@@ -24,5 +24,7 @@
   <xacro:arg name="can_fd" default="true" />
   <xacro:openarm_robot
-  arm_type="$(arg arm_type)" body_type="$(arg body_type)" joint_limits="${xacro.load_yaml('$(find openarm_description)/config/arm/$(arg arm_type)/joint_limits.yaml')}"
+  arm_type="$(arg arm_type)"
+  body_type="$(arg body_type)"
+  joint_limits="${xacro.load_yaml('$(find openarm_description)/config/arm/$(arg arm_type)/joint_limits.yaml')}"
   control_gains="${xacro.load_yaml('$(find openarm_description)/config/arm/$(arg arm_type)/control_gains.yaml')}"
   inertials="${xacro.load_yaml('$(find openarm_description)/config/arm/$(arg arm_type)/inertials.yaml')}"
@@ -36,5 +38,7 @@
   ee_kinematics="${xacro.load_yaml('$(find openarm_description)/config/ee/' + auto_ee_type + '/kinematics.yaml')}"
   ee_kinematics_link="${xacro.load_yaml('$(find openarm_description)/config/ee/' + auto_ee_type + '/kinematics_link.yaml')}"
-  ee_type="${auto_ee_type}" ros2_control="$(arg ros2_control)"
+  ee_joints_limits="${xacro.load_yaml('$(find openarm_description)/config/ee/' + auto_ee_type + '/joint_limits.yaml')}"
+  ee_type="${auto_ee_type}"
+  ros2_control="$(arg ros2_control)"
   can_interface="$(arg can_interface)"
   left_can_interface="$(arg left_can_interface)"

File: urdf/robot/v20/v20.urdf.xacro (robot description, xacro)
@@ -38,4 +38,5 @@
   ee_kinematics_link="${xacro.load_yaml('$(find openarm_description)/config/ee/' + auto_ee_type + '/kinematics_link.yaml')}"
   ee_inertials="${xacro.load_yaml('$(find openarm_description)/config/ee/' + auto_ee_type + '/inertials.yaml')}"
+  ee_joints_limits="${xacro.load_yaml('$(find openarm_description)/config/ee/' + auto_ee_type + '/joint_limits.yaml')}"
   ee_type="${auto_ee_type}"
   ros2_control="$(arg ros2_control)"

File: urdf/ros2_control/openarm.bimanual.ros2_control.xacro (robot description, xacro)
@@ -9,4 +9,5 @@
              fake_sensor_commands:=^|false
              hand:=^|false
+             ee_type:=^|parallel_link
              left_arm_prefix:=^|left_
              right_arm_prefix:=^|right_
@@ -22,9 +23,10 @@
           </xacro:if>
           <xacro:unless value="${use_fake_hardware}">
-            <plugin>openarm_hardware/OpenArm_v10HW</plugin>
+            <plugin>openarm_hardware/OpenArmHW</plugin>
             <param name="can_interface">${left_can_interface}</param>
             <param name="arm_prefix">${left_arm_prefix}</param>
             <param name="hand">${hand}</param>
             <param name="can_fd">${can_fd}</param>
+            <param name="ee_type">${ee_type}</param>
             <param name="kp1">${control_gains['joint1']['kp']}</param>
             <param name="kp2">${control_gains['joint2']['kp']}</param>
@@ -80,5 +82,5 @@
           </xacro:if>
           <xacro:unless value="${use_fake_hardware}">
-            <plugin>openarm_hardware/OpenArm_v10HW</plugin>
+            <plugin>openarm_hardware/OpenArmHW</plugin>
             <param name="can_interface">${right_can_interface}</param>
             <param name="arm_prefix">${right_arm_prefix}</param>

File: urdf/ros2_control/openarm.ros2_control.xacro (robot description, xacro)
@@ -8,4 +8,5 @@
              fake_sensor_commands:=^|false
              hand:=^|false
+             ee_type:=^|parallel_link
              gazebo_effort:=^|false
              arm_prefix:=''
@@ -22,9 +23,10 @@
           </xacro:if>
           <xacro:if value="${use_fake_hardware == 0}">
-            <plugin>openarm_hardware/OpenArm_${arm_type}HW</plugin>
+            <plugin>openarm_hardware/OpenArmHW</plugin>
             <param name="can_interface">${can_interface}</param>
             <param name="arm_prefix">${arm_prefix}</param>
             <param name="hand">${hand}</param>
             <param name="can_fd">${can_fd}</param>
+            <param name="ee_type">${ee_type}</param>
             <param name="kp1">${control_gains['joint1']['kp']}</param>
             <param name="kp2">${control_gains['joint2']['kp']}</param>
