Commit message: fix: body name

File: urdf/body/openarm_body.xacro (robot description, xacro)
@@ -13,5 +13,6 @@
               kinematics
               kinematics_link">
-    <xacro:property name="prefix" value="${'' if no_prefix else body_prefix + body_type + '_body_'}" />
+    <!-- <xacro:property name="prefix" value="${'' if no_prefix else body_prefix + 'body_'}" /> -->
+    <xacro:property name="prefix" value="${'' if no_prefix else 'openarm_' + 'body_'}" />
     <xacro:unless value="${not connected_to}">
     <link name="${connected_to}" />

File: urdf/body/openarm_body_macro.xacro (robot description, xacro)
@@ -32,5 +32,6 @@
   <!-- ========================================================== -->
   <xacro:macro name="body_link_with_sc" params="name no_prefix:='false' rpy:='0 0 0' kinematics_link">
-    <xacro:property name="prefix" value="${'' if no_prefix else body_prefix + body_type + '_'}" />
+    <!-- <xacro:property name="prefix" value="${'' if no_prefix else body_prefix + body_type + '_'}" /> -->
+    <xacro:property name="prefix" value="${'' if no_prefix else 'openarm' + '_' + body_prefix}" />
     <link name="${prefix}${name}">
       <visual name="${prefix}${name}_visual">

File: urdf/robot/openarm_robot.xacro (robot description, xacro)
@@ -63,5 +63,5 @@
         no_prefix="false"
         description_pkg="openarm_description"
-        connected_to="${body_type}_body_link0"
+        connected_to="openarm_body_link0"
         xyz="${left_arm_base_xyz}"
         rpy="${left_arm_base_rpy}"
@@ -88,5 +88,5 @@
         no_prefix="false"
         description_pkg="openarm_description"
-        connected_to="${body_type}_body_link0"
+        connected_to="openarm_body_link0"
         xyz="${right_arm_base_xyz}"
         rpy="${right_arm_base_rpy}"
