Commit message: fix: phsical parameter

File: urdf/arm/openarm_macro.xacro (robot description, xacro)
@@ -20,5 +20,5 @@
     </xacro:if>
   </xacro:macro>
-  <xacro:macro name="link_with_sc" params="name no_prefix:='false' rpy:='0 0 0' kinematics_link:=''  reflect:=1">
+  <xacro:macro name="link_with_sc" params="name no_prefix:='false' rpy:='0 0 0' kinematics_link:='' reflect:=1 inertials:=^">
     <!-- <xacro:property name="prefix" value="${'' if no_prefix else arm_prefix + arm_type + '_'}" /> -->
     <xacro:property name="prefix" value="${'' if no_prefix else 'openarm' + '_' +  arm_prefix}" />

File: urdf/robot/v10.urdf.xacro (robot description, xacro)
@@ -11,11 +11,7 @@
   </xacro:if>
   <xacro:arg name="parent" default="world" />
-  <!-- If `gazebo` arg is set and `parent` not empty, what position offset between `parent` & $(arm_type)_link0 -->
   <xacro:arg name="xyz" default="0 0 0" />
-  <!-- If `gazebo` arg is set and `parent` not empty, what rotation offset between `parent` & $(arm_type)_link0 -->
   <xacro:arg name="rpy" default="0 0 0" />
-  <!-- Is the robot being controlled with ros2_control?" -->
   <xacro:arg name="ros2_control" default="false" />
-  <!-- IP address or hostname of the robot" -->
   <xacro:arg name="can_interface" default="can0" />
   <xacro:arg name="left_can_interface" default="can1" />
@@ -23,11 +19,7 @@
   <xacro:arg name="left_arm_prefix" default="left_" />
   <xacro:arg name="right_arm_prefix" default="right_" />
-  <!-- Should a fake hardware be used? -->
   <xacro:arg name="use_fake_hardware" default="false" />
-  <!-- Should fake sensors be used? -->
   <xacro:arg name="fake_sensor_commands" default="false" />
-  <!-- For a multi arm setup, we need a threaded robot running async-->
   <xacro:arg name="bimanual" default="false" />
-  <!-- used in bimanual -->
   <xacro:arg name="right_arm_base_xyz" default="0.0 -0.031 0.698" />
   <xacro:arg name="right_arm_base_rpy" default="1.5708 0 0" />
