Commit message: Remove tracked files now listed in .gitignore

File: urdf/arm/openarm_arm.xacro (robot description, xacro)
@@ -86,10 +86,10 @@
       <xacro:openarm-limits name="joint6" config="${joint_limits}" />
     </joint>
-    <xacro:link_with_sc no_prefix="${no_prefix}" name="link7" rpy="0 0 0"  kinematics_link="${kinematics_link}" reflect="${reflect}"/>
+    <xacro:link_with_sc no_prefix="${no_prefix}" name="link7" kinematics_link="${kinematics_link}" reflect="${reflect}"/>
     <joint name="${prefix}joint7" type="revolute">
       <xacro:openarm-kinematics name="joint7" config="${kinematics}" />
       <parent link="${prefix}link6"/>
       <child link="${prefix}link7"/>
-      <axis xyz="0 1 0"/>
+      <axis xyz="0 -1 0"/>
       <xacro:openarm-limits name="joint7" config="${joint_limits}" />
     </joint>

File: urdf/ee/openarm_hand_macro.xacro (robot description, xacro)
@@ -21,5 +21,4 @@
   </xacro:macro>
   <xacro:macro name="ee_link_with_sc" params="name prefix rpy:='0 0 0' ee_kinematics_link">
-    <!-- sub-link defining detailed meshes for collision with environment -->
     <link name="${prefix}${name}">
       <visual name="${prefix}${name}_visual">

Commit message: Fix joint 7 right hand rule

File: urdf/arm/openarm_arm.xacro (robot description, xacro)
@@ -91,5 +91,5 @@
       <parent link="${prefix}link6"/>
       <child link="${prefix}link7"/>
-      <axis xyz="0 -1 0"/>
+      <axis xyz="0 ${reflect} 0"/>
       <xacro:openarm-limits name="joint7" config="${joint_limits}" />
     </joint>

Commit message: delete: comment

File: urdf/arm/openarm_arm.xacro (robot description, xacro)
@@ -2,12 +2,5 @@
 <robot xmlns:xacro="http://www.ros.org/wiki/xacro" name="openarm">
   <xacro:include filename="$(find openarm_description)/urdf/arm/openarm_macro.xacro" />
-  <!-- arm_type: Namespace of the robot arm. Serves to differentiate between arms in case of multiple instances. -->
-  <!-- joint_limits: description of the joint limits that comes from a YAML file. Example definition: ${xacro.load_yaml('$(find openarm_description)/robots/fr3/joint_limits.yaml')} -->
-  <!-- kinematics: description of the kinematics that comes from a YAML file. Example definition: ${xacro.load_yaml('$(find openarm_description)/robots/fr3/kinematics.yaml')} -->
-  <!-- inertials: description of the inertials that comes from a YAML file. Example definition: ${xacro.load_yaml('$(find openarm_description)/robots/fr3/inertials.yaml')} -->
   <xacro:macro name="openarm_arm" params="arm_type arm_prefix:='' no_prefix:=false description_pkg:='openarm_description' connected_to:='base' xyz:='0 0 0' rpy:='0 0 0' joint_limits inertials kinematics kinematics_link kinematics_offset:=none " >
-    <!-- Define a property that defaults to 'arm_prefix_arm_type' concatenated with an underscore if 'no_prefix' is not set -->
-    <!-- <xacro:property name="prefix" value="${'' if no_prefix else arm_prefix + arm_type + '_'}" /> -->
-    <!-- <xacro:property name="prefix" value="${'' if no_prefix else arm_prefix + 'openarm' + '_'}" /> -->
     <xacro:property name="prefix" value="${'' if no_prefix else 'openarm' + '_' + arm_prefix}" />
     <xacro:if value="${arm_prefix == 'right_'}">
@@ -17,10 +10,5 @@
       <xacro:property name="reflect" value="-1" />
     </xacro:unless>
-    <!-- <xacro:if value="${gazebo}">
-      <xacro:property name="connected_to" value="" />
-    </xacro:if> -->
     <xacro:unless value="${connected_to == ''}">
-      <!-- <link name="${connected_to}">
-      </link> -->
       <joint name="${prefix}${connected_to}_joint" type="fixed">
         <parent link="${connected_to}"/>

File: urdf/arm/openarm_macro.xacro (robot description, xacro)
@@ -1,10 +1,4 @@
 <?xml version="1.0"?>
 <robot xmlns:xacro="http://www.ros.org/wiki/xacro">
-  <!-- ============================================================== -->
-  <!-- Macro to add an <inertial> tag based on yaml-load properties   -->
-  <!--                                                                -->
-  <!-- name:     Name of the robot link (without prefix)              -->
-  <!-- inertial: Dictionary of inertia properties (see inertial.yaml) -->
-  <!-- ============================================================== -->
   <xacro:macro name="openarm-inertials" params="name inertials:=^ reflect:=1">
     <xacro:unless value="${name in inertials}">
@@ -26,14 +20,4 @@
     </xacro:if>
   </xacro:macro>
-  <!-- ========================================================== -->
-  <!-- Macro to add a single link, both with                      -->
-  <!--  * detailed meshes for environmental collision checking    -->
-  <!--  * and coarse geometry models for self-collision checking  -->
-  <!--    (only if 'gazebo' param is set)                         -->
-  <!--                                                            -->
-  <!-- name:  Name of the robot link (without prefix)             -->
-  <!-- rpy:   Rotation of the *_sc link relative to parent [rad]  -->
-  <!-- self_collision_geometries:  self <collision> models        -->
-  <!-- ========================================================== -->
   <xacro:macro name="link_with_sc" params="name no_prefix:='false' rpy:='0 0 0' kinematics_link:=''  reflect:=1">
     <!-- <xacro:property name="prefix" value="${'' if no_prefix else arm_prefix + arm_type + '_'}" /> -->
@@ -56,52 +40,4 @@
     </link>
   </xacro:macro>
-  <!-- ========================================================== -->
-  <!-- Adds the required tags to simulate one joint in gazebo     -->
-  <!--                                                            -->
-  <!-- joint - Name of the openarm joint to simulate                  -->
-  <!-- transmission - type of the transmission of the joint       -->
-  <!-- ========================================================== -->
-  <!-- <xacro:macro name="gazebo-joint" params="joint transmission:=hardware_interface/EffortJointInterface">
-    <gazebo reference="${joint}">
-      <provideFeedback>true</provideFeedback>
-    </gazebo>
-    <transmission name="${joint}_transmission">
-      <type>transmission_interface/SimpleTransmission</type>
-      <joint name="${joint}">
-        <hardwareInterface>${transmission}</hardwareInterface>
-      </joint>
-      <actuator name="${joint}_motor">
-        <hardwareInterface>${transmission}</hardwareInterface>
-      </actuator>
-    </transmission>
-  </xacro:macro> -->
-  <!-- <xacro:macro name="gazebo-friction" params="link mu">
-    <gazebo reference="${link}">
-      <collision>
-        <max_contacts>10</max_contacts>
-        <surface>
-          <contact>
-            <ode>
-              <max_vel>0</max_vel>
-              <min_depth>0.001</min_depth>
-            </ode>
-          </contact>
-          <friction>
-            <ode>
-              <mu>${mu}</mu>
-              <mu2>${mu}</mu2>
-            </ode>
-          </friction>
-          <bounce/>
-        </surface>
-      </collision>
-    </gazebo>
-  </xacro:macro> -->
-  <!-- ========================================================== -->
-  <!-- Adds the required tags to provide a `openarmStateInterface` -->
-  <!-- when simulating with openarm_hw_sim plugin                  -->
-  <!--                                                            -->
-  <!-- arm_type - Arm ID of the fer to simulate (default 'fer')     -->
-  <!-- ========================================================== -->
   <xacro:macro name="transmission-openarm-state" params="arm_type:=fer">
     <transmission name="${arm_prefix}${arm_type}_openarm_state">
@@ -123,12 +59,4 @@
     </transmission>
   </xacro:macro>
-  <!-- ============================================================ -->
-  <!-- Adds the required tags to provide a `openarmModelInterface`   -->
-  <!-- when simulating with openarm_hw_sim plugin                    -->
-  <!--                                                              -->
-  <!-- arm_type - Arm ID of the fer to simulate (default 'fer')       -->
-  <!-- root   - Joint name of the base of the robot                 -->
-  <!-- tip    - Joint name of the tip of the robot (flange or hand) -->
-  <!-- ============================================================ -->
   <xacro:macro name="transmission-openarm-model" params="arm_type:=v10 root:=v10_joint1 tip:=v10_joint7">
     <transmission name="${arm_prefix}${arm_type}_openarm_model">
@@ -154,11 +82,4 @@
     </inertial>
   </xacro:macro>
-  <!-- ========================================================================= -->
-  <!-- Adds the <limit ... /> & <safety_controller/> tags given a config file    -->
-  <!-- of joint limits                                                           -->
-  <!--                                                                           -->
-  <!-- config - YAML struct defining joint limits (e.g. fer/joint_limits.yaml)   -->
-  <!-- name   - Name of the joint for which to add limits to                     -->
-  <!-- ========================================================================= -->
   <xacro:macro name="openarm-limits" params="name config reflect:=1 offset:=0">
     <xacro:property name="limits" value="${config[name]['limit']}"/>
@@ -181,10 +102,4 @@
       velocity="${limits.velocity}" />
   </xacro:macro>
-  <!-- ========================================================================= -->
-  <!-- Adds the <kinematics ... /> tag given a config file of joint kinematics   -->
-  <!--                                                                           -->
-  <!-- config - YAML struct defining joint kinematics (e.g. fer/kinematics.yaml) -->
-  <!-- name   - Name of the joint for which to add kinematics to                 -->
-  <!-- ========================================================================= -->
   <xacro:macro name="openarm-kinematics" params="name config offset:=none reflect:=1">
     <xacro:property name="kinematics" value="${config[name]['kinematic']}" lazy_eval="false" />

File: urdf/body/openarm_body_macro.xacro (robot description, xacro)
@@ -1,10 +1,4 @@
 <?xml version="1.0"?>
 <robot xmlns:xacro="http://www.ros.org/wiki/xacro">
-  <!-- ============================================================== -->
-  <!-- Macro to add an <inertial> tag based on yaml-load properties   -->
-  <!--                                                                -->
-  <!-- name:     Name of the robot link (without prefix)              -->
-  <!-- inertial: Dictionary of inertia properties (see inertial.yaml) -->
-  <!-- ============================================================== -->
   <xacro:macro name="openarm-body-inertials" params="name inertials:=^">
       <xacro:unless value="${name in inertials}">${xacro.warning('No inertia properties defined for: ' + name)}</xacro:unless>
@@ -22,13 +16,4 @@
       </xacro:if>
   </xacro:macro>
-  <!-- ========================================================== -->
-  <!-- Macro to add a single link, both with                      -->
-  <!--  * detailed meshes for environmental collision checking    -->
-  <!--  * and coarse geometry models for self-collision checking  -->
-  <!--                                                            -->
-  <!-- name:  Name of the robot link (without prefix)             -->
-  <!-- rpy:   Rotation of the *_sc link relative to parent [rad]  -->
-  <!-- self_collision_geometries:  self <collision> models        -->
-  <!-- ========================================================== -->
   <xacro:macro name="body_link_with_sc" params="name no_prefix:='false' rpy:='0 0 0' kinematics_link">
     <!-- <xacro:property name="prefix" value="${'' if no_prefix else body_prefix + body_type + '_'}" /> -->

File: urdf/robot/openarm_robot.xacro (robot description, xacro)
@@ -174,66 +174,5 @@
         </xacro:if>
         </xacro:if>
-        <!-- <xacro:if value="${hand and ee_type != 'none' and ee_type != 'openarm_hand'}">
-        <xacro:property name="special_connection" value="$(arg special_connection)" />
-        <xacro:property name="connection" value="${special_connection if special_connection == '' else arm_type + '_link8'}" />
-        <xacro:ee_with_one_link
-            connected_to="${arm_prefix_modified}${connection}"
-            arm_type="${arm_type}"
-            arm_prefix="${arm_prefix_modified}"
-            ee_type="${ee_type}"
-            ee_inertials="${xacro.load_yaml('$(find openarm_description)/config/hand/$(arg ee_type)_inertials.yaml')}"
-            ee_kinematics_link="${xacro.load_yaml('$(find openarm_description)/config/hand/openarm_hand/kinematics_link.yaml')}"
-            rpy_ee="$(arg rpy_ee)"
-            xyz_ee="$(arg xyz_ee)"
-            tcp_xyz="$(arg tcp_xyz)"
-            tcp_rpy="$(arg tcp_rpy)"
-            description_pkg="$(arg description_pkg)"
-        />
-        </xacro:if> -->
         </xacro:if>
-        <!-- <xacro:if value="${gazebo}">
-        <xacro:if value="${parent != ''}">
-            <xacro:if value="${parent == 'world'}">
-            <link name="${parent}" />
-            </xacro:if>
-            <joint name="${parent}_joint" type="fixed">
-            <origin xyz="${xyz}" rpy="${rpy}" />
-            <parent link="${parent}" />
-            <child  link="${arm_type}_link0" />
-            </joint>
-        </xacro:if> -->
-        <!-- <xacro:gazebo-joint joint="${arm_type}_joint1" transmission="hardware_interface/PositionJointInterface" />
-        <xacro:gazebo-joint joint="${arm_type}_joint2" transmission="hardware_interface/PositionJointInterface" />
-        <xacro:gazebo-joint joint="${arm_type}_joint3" transmission="hardware_interface/PositionJointInterface" />
-        <xacro:gazebo-joint joint="${arm_type}_joint4" transmission="hardware_interface/PositionJointInterface" />
-        <xacro:gazebo-joint joint="${arm_type}_joint5" transmission="hardware_interface/PositionJointInterface" />
-        <xacro:gazebo-joint joint="${arm_type}_joint6" transmission="hardware_interface/PositionJointInterface" />
-        <xacro:gazebo-joint joint="${arm_type}_joint7" transmission="hardware_interface/PositionJointInterface" />
-        <xacro:gazebo-joint joint="${arm_type}_joint1" transmission="hardware_interface/VelocityJointInterface" />
-        <xacro:gazebo-joint joint="${arm_type}_joint2" transmission="hardware_interface/VelocityJointInterface" />
-        <xacro:gazebo-joint joint="${arm_type}_joint3" transmission="hardware_interface/VelocityJointInterface" />
-        <xacro:gazebo-joint joint="${arm_type}_joint4" transmission="hardware_interface/VelocityJointInterface" />
-        <xacro:gazebo-joint joint="${arm_type}_joint5" transmission="hardware_interface/VelocityJointInterface" />
-        <xacro:gazebo-joint joint="${arm_type}_joint6" transmission="hardware_interface/VelocityJointInterface" />
-        <xacro:gazebo-joint joint="${arm_type}_joint7" transmission="hardware_interface/VelocityJointInterface" />
-        <xacro:gazebo-joint joint="${arm_type}_joint1" transmission="hardware_interface/EffortJointInterface" />
-        <xacro:gazebo-joint joint="${arm_type}_joint2" transmission="hardware_interface/EffortJointInterface" />
-        <xacro:gazebo-joint joint="${arm_type}_joint3" transmission="hardware_interface/EffortJointInterface" />
-        <xacro:gazebo-joint joint="${arm_type}_joint4" transmission="hardware_interface/EffortJointInterface" />
-        <xacro:gazebo-joint joint="${arm_type}_joint5" transmission="hardware_interface/EffortJointInterface" />
-        <xacro:gazebo-joint joint="${arm_type}_joint6" transmission="hardware_interface/EffortJointInterface" />
-        <xacro:gazebo-joint joint="${arm_type}_joint7" transmission="hardware_interface/EffortJointInterface" />  -->
-        <!-- <xacro:transmission-openarm-state arm_type="${arm_type}" />
-        <xacro:transmission-openarm-model arm_type="${arm_type}"
-            root="${arm_type}_joint1"
-            tip="${arm_type}_joint8"
-        /> -->
-        <!-- <xacro:if value="${ee_type == 'openarm_hand'}">
-            <xacro:gazebo-joint joint="${arm_type}_finger_joint1" transmission="hardware_interface/EffortJointInterface" />
-            <xacro:gazebo-joint joint="${arm_type}_finger_joint2" transmission="hardware_interface/EffortJointInterface" />
-            <xacro:gazebo-friction link="${arm_type}_leftfinger" mu="1.13" />
-            <xacro:gazebo-friction link="${arm_type}_rightfinger" mu="1.13" />
-        </xacro:if>
-        </xacro:if> -->
   </xacro:macro>
 </robot>

File: urdf/robot/v10.urdf.xacro (robot description, xacro)
@@ -2,20 +2,12 @@
 <robot xmlns:xacro="http://www.ros.org/wiki/xacro" name="openarm">
   <xacro:include filename="$(find openarm_description)/urdf/robot/openarm_robot.xacro"/>
-  <!--
-    DEPRECATION NOTICE
-    argument arm_type is no longer supported and will be removed in the future.
-    This argument is ignored.
-  -->
   <xacro:arg name="arm_type" default="v10" />
   <xacro:arg name="body_type" default="v10" />
   <xacro:arg name="ee_type" default="openarm_hand" />
-  <!-- Don't print a prefix for joints, visuals, and links? -->
   <xacro:arg name="no_prefix" default="false"/>
-  <!-- Should an end-effector be mounted at the flange?" -->
   <xacro:arg name="hand" default="true" />
   <xacro:if value="$(eval ee_type == 'none')">
     <xacro:property name="hand" value="false"/>
   </xacro:if>
-  <!-- If `gazebo` arg is set, to which frame shall $(arm_type)_link0 be parented. Empty string for not fixing at all -->
   <xacro:arg name="parent" default="world" />
   <!-- If `gazebo` arg is set and `parent` not empty, what position offset between `parent` & $(arm_type)_link0 -->
@@ -35,6 +27,4 @@
   <!-- Should fake sensors be used? -->
   <xacro:arg name="fake_sensor_commands" default="false" />
-  <!-- Should the robot be spawned in Gazebo with effort interfaces?" -->
-  <!-- <xacro:arg name="gazebo_effort" default="false" /> -->
   <!-- For a multi arm setup, we need a threaded robot running async-->
   <xacro:arg name="bimanual" default="false" />
