Commit message: fix: arm config path

File: urdf/arm/openarm_arm.xacro (robot description, xacro)
@@ -17,6 +17,6 @@
       </joint>
     </xacro:unless>
-    <xacro:link_with_sc no_prefix="${no_prefix}" name="link0" kinematics_link="${kinematics_link}" reflect="${reflect}"/>
-    <xacro:link_with_sc no_prefix="${no_prefix}" name="link1" kinematics_link="${kinematics_link}" reflect="${reflect}"/>
+    <xacro:link_with_sc no_prefix="${no_prefix}" name="link0" kinematics_link="${kinematics_link}" inertials="${inertials}" reflect="${reflect}"/>
+    <xacro:link_with_sc no_prefix="${no_prefix}" name="link1" kinematics_link="${kinematics_link}" inertials="${inertials}" reflect="${reflect}"/>
     <joint name="${prefix}joint1" type="revolute">
       <xacro:openarm-kinematics name="joint1" config="${kinematics}" reflect="${reflect}"/>
@@ -27,5 +27,5 @@
     </joint>
     <!-- for bimanual offset -->
-    <xacro:link_with_sc no_prefix="${no_prefix}" name="link2" kinematics_link="${kinematics_link}" reflect="${reflect}"/>
+    <xacro:link_with_sc no_prefix="${no_prefix}" name="link2" kinematics_link="${kinematics_link}" inertials="${inertials}" reflect="${reflect}"/>
     <xacro:property name="limit_offset_joint2" value="0" />
     <xacro:if value="${prefix.find('right_') != -1}">
@@ -42,5 +42,5 @@
       <xacro:openarm-limits name="joint2" config="${joint_limits}" reflect="${reflect}" offset="${limit_offset_joint2}"/>
     </joint>
-    <xacro:link_with_sc no_prefix="${no_prefix}" name="link3" kinematics_link="${kinematics_link}" reflect="${reflect}"/>
+    <xacro:link_with_sc no_prefix="${no_prefix}" name="link3" kinematics_link="${kinematics_link}" inertials="${inertials}" reflect="${reflect}"/>
     <joint name="${prefix}joint3" type="revolute">
       <xacro:openarm-kinematics name="joint3" config="${kinematics}" />
@@ -58,5 +58,5 @@
       <xacro:openarm-limits name="joint4" config="${joint_limits}" />
     </joint>
-    <xacro:link_with_sc no_prefix="${no_prefix}" name="link5" kinematics_link="${kinematics_link}" reflect="${reflect}" />
+    <xacro:link_with_sc no_prefix="${no_prefix}" name="link5" kinematics_link="${kinematics_link}" inertials="${inertials}" reflect="${reflect}" />
     <joint name="${prefix}joint5" type="revolute">
       <xacro:openarm-kinematics name="joint5" config="${kinematics}" />
@@ -66,5 +66,5 @@
       <xacro:openarm-limits name="joint5" config="${joint_limits}" />
     </joint>
-    <xacro:link_with_sc no_prefix="${no_prefix}" name="link6" kinematics_link="${kinematics_link}" reflect="${reflect}"/>
+    <xacro:link_with_sc no_prefix="${no_prefix}" name="link6" kinematics_link="${kinematics_link}" inertials="${inertials}" reflect="${reflect}"/>
     <joint name="${prefix}joint6" type="revolute">
       <xacro:openarm-kinematics name="joint6" config="${kinematics}" />
@@ -74,5 +74,5 @@
       <xacro:openarm-limits name="joint6" config="${joint_limits}" />
     </joint>
-    <xacro:link_with_sc no_prefix="${no_prefix}" name="link7" kinematics_link="${kinematics_link}" reflect="${reflect}"/>
+    <xacro:link_with_sc no_prefix="${no_prefix}" name="link7" kinematics_link="${kinematics_link}" inertials="${inertials}" reflect="${reflect}"/>
     <joint name="${prefix}joint7" type="revolute">
       <xacro:openarm-kinematics name="joint7" config="${kinematics}" />

File: urdf/arm/openarm_macro.xacro (robot description, xacro)
@@ -37,5 +37,5 @@
         </geometry>
       </collision>
-      <xacro:openarm-inertials name="${name}" />
+      <xacro:openarm-inertials name="${name}" inertials="${inertials}" reflect="${reflect}" />
     </link>
   </xacro:macro>

File: urdf/robot/v10.urdf.xacro (robot description, xacro)
@@ -29,9 +29,9 @@
   arm_type="v10"
   body_type="v10"
-  joint_limits="${xacro.load_yaml('$(find openarm_description)/config/v10/joint_limits.yaml')}"
-  inertials="${xacro.load_yaml('$(find openarm_description)/config/v10/inertials.yaml')}"
-  kinematics="${xacro.load_yaml('$(find openarm_description)/config/v10/kinematics.yaml')}"
-  kinematics_link="${xacro.load_yaml('$(find openarm_description)/config/v10/kinematics_link.yaml')}"
-  kinematics_offset="${xacro.load_yaml('$(find openarm_description)/config/v10/kinematics_offset.yaml')}"
+  joint_limits="${xacro.load_yaml('$(find openarm_description)/config//arm/v10/joint_limits.yaml')}"
+  inertials="${xacro.load_yaml('$(find openarm_description)/config/arm/v10/inertials.yaml')}"
+  kinematics="${xacro.load_yaml('$(find openarm_description)/config/arm/v10/kinematics.yaml')}"
+  kinematics_link="${xacro.load_yaml('$(find openarm_description)/config/arm/v10/kinematics_link.yaml')}"
+  kinematics_offset="${xacro.load_yaml('$(find openarm_description)/config/arm/v10/kinematics_offset.yaml')}"
   body_inertials="${xacro.load_yaml('$(find openarm_description)/config/body/v10/inertials.yaml')}"
   body_kinematics="${xacro.load_yaml('$(find openarm_description)/config/body/v10/kinematics.yaml')}"

File: urdf/robot/v10_bimanual.urdf (robot description, URDF)
Before this commit: robot openarm, 28 links, 27 joints
Links:
- link openarm_left_link4: mass 1.3699337287025453 -> 0.5598534566833373
- link openarm_left_link6: mass 0.3540202773187987 -> 0.385202773187987
- link openarm_left_link7: mass 0.5499771327380578 -> 0.3859771327380578
- link openarm_right_link4: mass 1.3699337287025453 -> 0.5598534566833373
- link openarm_right_link6: mass 0.3540202773187987 -> 0.385202773187987
- link openarm_right_link7: mass 0.5499771327380578 -> 0.3859771327380578
Joints:
- joint openarm_left_joint1: limit lower=-3.490659 upper=1.3962629999999998 effort=54 velocity=45 -> lower=-3.490659 upper=1.3962629999999998 effort=40 velocity=16.754666
- joint openarm_left_joint2: limit lower=-3.3161253267948965 upper=0.17453267320510335 effort=54 velocity=45 -> lower=-3.3161253267948965 upper=0.17453267320510335 effort=40 velocity=16.754666
- joint openarm_left_joint3: limit lower=-1.570796 upper=1.570796 effort=28 velocity=8 -> lower=-1.570796 upper=1.570796 effort=27 velocity=5.445426
- joint openarm_left_joint4: limit lower=0.0 upper=2.443461 effort=28 velocity=8 -> lower=0.0 upper=2.443461 effort=27 velocity=5.445426
- joint openarm_left_joint5: limit lower=-1.570796 upper=1.570796 effort=10 velocity=30 -> lower=-1.570796 upper=1.570796 effort=7 velocity=20.943946
- joint openarm_left_joint6: limit lower=-0.785398 upper=0.785398 effort=10 velocity=30 -> lower=-0.785398 upper=0.785398 effort=7 velocity=20.943946
- joint openarm_left_joint7: limit lower=-1.570796 upper=1.570796 effort=10 velocity=30 -> lower=-1.570796 upper=1.570796 effort=7 velocity=20.943946
- joint openarm_right_joint1: limit lower=-1.396263 upper=3.490659 effort=54 velocity=45 -> lower=-1.396263 upper=3.490659 effort=40 velocity=16.754666
- joint openarm_right_joint2: limit lower=-0.17453267320510335 upper=3.3161253267948965 effort=54 velocity=45 -> lower=-0.17453267320510335 upper=3.3161253267948965 effort=40 velocity=16.754666
- joint openarm_right_joint3: limit lower=-1.570796 upper=1.570796 effort=28 velocity=8 -> lower=-1.570796 upper=1.570796 effort=27 velocity=5.445426
- joint openarm_right_joint4: limit lower=0.0 upper=2.443461 effort=28 velocity=8 -> lower=0.0 upper=2.443461 effort=27 velocity=5.445426
- joint openarm_right_joint5: limit lower=-1.570796 upper=1.570796 effort=10 velocity=30 -> lower=-1.570796 upper=1.570796 effort=7 velocity=20.943946
- joint openarm_right_joint6: limit lower=-0.785398 upper=0.785398 effort=10 velocity=30 -> lower=-0.785398 upper=0.785398 effort=7 velocity=20.943946
- joint openarm_right_joint7: limit lower=-1.570796 upper=1.570796 effort=10 velocity=30 -> lower=-1.570796 upper=1.570796 effort=7 velocity=20.943946
