Commit message: refactor: remove hand intermediate link and unify end-effector structure

File: urdf/arm/openarm_arm.xacro (robot description, xacro)
@@ -82,10 +82,4 @@
       <xacro:openarm-limits name="joint7" config="${joint_limits}" />
     </joint>
-    <!-- <link name="${prefix}link8"/>
-    <joint name="${prefix}joint8" type="fixed">
-      <xacro:openarm-kinematics name="joint8" config="${kinematics}" />
-      <parent link="${prefix}link7" />
-      <child link="${prefix}link8" />
-    </joint> -->
   </xacro:macro>
 </robot>

File: urdf/ee/ee_dispatcher.xacro (robot description, xacro)
@@ -1,9 +1,9 @@
 <?xml version='1.0' encoding='utf-8'?>
 <robot xmlns:xacro="http://www.ros.org/wiki/xacro">
-  <xacro:include filename="$(find openarm_description)/urdf/ee/parallel_link/openarm_hand.xacro" />
-  <xacro:include filename="$(find openarm_description)/urdf/ee/pinch_gripper/openarm_v20_hand.xacro" />
+  <xacro:include filename="$(find openarm_description)/urdf/ee/parallel_link/openarm_parallel_gripper.xacro" />
+  <xacro:include filename="$(find openarm_description)/urdf/ee/pinch_gripper/openarm_v20_pinch_gripper.xacro" />
   <xacro:macro name="openarm_ee" params="ee_type connected_to arm_type arm_prefix ee_kinematics_link ee_inertials">
     <xacro:if value="${ee_type == 'parallel_link'}">
-      <xacro:openarm_hand
+      <xacro:openarm_parallel_gripper
         connected_to="${connected_to}"
         arm_type="${arm_type}"
@@ -15,5 +15,5 @@
     </xacro:if>
     <xacro:if value="${ee_type == 'pinch_gripper'}">
-      <xacro:openarm_v20_hand
+      <xacro:openarm_v20_pinch_gripper
         connected_to="${connected_to}"
         arm_type="${arm_type}"

File: urdf/ee/parallel_link/openarm_parallel_gripper.xacro (robot description, xacro)
@@ -1,27 +1,13 @@
 <?xml version="1.0" encoding="utf-8"?>
-<robot xmlns:xacro="http://www.ros.org/wiki/xacro" name="hand">
-  <!-- safety_distance: Minimum safety distance in [m] by which the collision volumes are expanded and which is enforced during robot motions -->
-  <xacro:macro name="openarm_hand" params="connected_to:='' arm_type arm_prefix:='' ee_type ee_inertials ee_kinematics_link rpy_ee:='0 0 0' xyz_ee:='0 0 0' tcp_xyz:='0 0 0' tcp_rpy:='0 0 0' description_pkg:=openarm_description">
+<robot xmlns:xacro="http://www.ros.org/wiki/xacro" name="parallel_gripper">
+  <xacro:macro name="openarm_parallel_gripper" params="connected_to:='' arm_type arm_prefix:='' ee_type ee_inertials ee_kinematics_link rpy_ee:='0 0 0' xyz_ee:='0 0 0' tcp_xyz:='0 0 0' tcp_rpy:='0 0 0' description_pkg:=openarm_description">
     <xacro:property name="ee_prefix" default=""/>
     <xacro:unless value="${arm_type == ''}">
-      <!-- <xacro:property name="ee_prefix" value="${arm_prefix}${arm_type}_" /> -->
       <xacro:property name="ee_prefix" value="openarm_${arm_prefix}" />
     </xacro:unless>
-    <xacro:ee_link_with_sc name="hand" prefix="${ee_prefix}" ee_kinematics_link="${ee_kinematics_link}"/>
-    <!-- <link name="${ee_prefix}hand"/> -->
-    <xacro:unless value="${connected_to == ''}">
-      <!-- <joint name="${ee_prefix}hand_joint" type="fixed"> -->
-      <joint name="${arm_prefix}openarm_hand_joint" type="fixed">
-        <parent link="${connected_to}" />
-        <child link="${ee_prefix}hand" />
-        <origin xyz="${xyz_ee}" rpy="${rpy_ee}" />
-      </joint>
-    </xacro:unless>
-    <!-- Define the hand_tcp frame -->
     <link name="${ee_prefix}hand_tcp" />
     <joint name="${ee_prefix}hand_tcp_joint" type="fixed">
       <origin xyz="${tcp_xyz}" rpy="${tcp_rpy}" />
-      <parent link="${ee_prefix}hand" />
-      <child link="${ee_prefix}hand_tcp" />
+      <parent link="${connected_to}" /> <child link="${ee_prefix}hand_tcp" />
     </joint>
     <link name="${ee_prefix}left_finger">
@@ -56,6 +42,5 @@
     </link>
     <joint name="${ee_prefix}finger_joint1" type="prismatic">
-      <parent link="${ee_prefix}hand" />
-      <child link="${ee_prefix}right_finger" />
+      <parent link="${connected_to}" /> <child link="${ee_prefix}right_finger" />
       <origin xyz="0 -0.006 0.015" rpy="0 0 0" />
       <axis xyz="0 -1 0" />
@@ -63,6 +48,5 @@
     </joint>
     <joint name="${ee_prefix}finger_joint2" type="prismatic">
-      <parent link="${ee_prefix}hand" />
-      <child link="${ee_prefix}left_finger" />
+      <parent link="${connected_to}" /> <child link="${ee_prefix}left_finger" />
       <origin xyz="0 0.006 0.015" rpy="0 0 0" />
       <axis xyz="0 1 0" />

File: urdf/ee/pinch_gripper/openarm_v20_pinch_gripper.xacro (robot description, xacro)
@@ -1,5 +1,4 @@
 <?xml version="1.0" encoding="utf-8"?>
-<robot xmlns:xacro="http://www.ros.org/wiki/xacro" name="hand">
-  <xacro:macro name="openarm_v20_hand" params="connected_to:='' arm_type arm_prefix:='' ee_type ee_inertials ee_kinematics_link rpy_ee:='0 0 0' xyz_ee:='0 0 0' tcp_xyz:='0 0 0' tcp_rpy:='0 0 0' description_pkg:=openarm_description">
+<robot xmlns:xacro="http://www.ros.org/wiki/xacro" name="pinch_gripper"> <xacro:macro name="openarm_v20_pinch_gripper" params="connected_to:='' arm_type arm_prefix:='' ee_type ee_inertials ee_kinematics_link rpy_ee:='0 0 0' xyz_ee:='0 0 0' tcp_xyz:='0 0 0' tcp_rpy:='0 0 0' description_pkg:=openarm_description">
     <xacro:property name="ee_prefix" value=""/>
     <xacro:unless value="${arm_type == ''}">
@@ -7,22 +6,9 @@
     </xacro:unless>
     <xacro:property name="reflect" value="${-1 if arm_prefix == 'left_' else 1}" />
-    <!-- hand link -->
-    <xacro:ee_link_with_sc name="hand" prefix="${ee_prefix}" ee_kinematics_link="${ee_kinematics_link}" reflect="${reflect}"/>
-    <!-- hand joint -->
-    <xacro:unless value="${connected_to == ''}">
-      <joint name="${arm_prefix}openarm_hand_joint" type="fixed">
-        <parent link="${connected_to}" />
-        <child link="${ee_prefix}hand" />
-        <origin xyz="${xyz_ee}" rpy="${rpy_ee}" />
-      </joint>
-    </xacro:unless>
-    <!-- tcp frame -->
     <link name="${ee_prefix}hand_tcp" />
     <joint name="${ee_prefix}hand_tcp_joint" type="fixed">
       <origin xyz="${tcp_xyz}" rpy="${tcp_rpy}" />
-      <parent link="${ee_prefix}hand" />
-      <child link="${ee_prefix}hand_tcp" />
+      <parent link="${connected_to}" /> <child link="${ee_prefix}hand_tcp" />
     </joint>
-    <!-- finger links -->
     <xacro:ee_finger_link_with_sc
         name="right_finger"
@@ -39,17 +25,12 @@
         finger_reflect="1"
     />
-    <!-- finger joints -->
     <joint name="${ee_prefix}finger_joint1" type="revolute">
-      <parent link="${ee_prefix}hand" />
-      <child link="${ee_prefix}right_finger" />
-      <origin xyz="0 0.006 0.015" rpy="0 0 0" />
-      <axis xyz="0 1 0" />
+      <parent link="${connected_to}" /> <child link="${ee_prefix}right_finger" />
+      <origin xyz="0 0.006 0.015" rpy="0 0 0" /> <axis xyz="0 1 0" />
       <limit effort="333" lower="0.0" upper="1.5708" velocity="10.0" />
     </joint>
     <joint name="${ee_prefix}finger_joint2" type="revolute">
-      <parent link="${ee_prefix}hand" />
-      <child link="${ee_prefix}left_finger" />
-      <origin xyz="0 -0.006 0.015" rpy="0 0 0" />
-      <axis xyz="0 -1 0" />
+      <parent link="${connected_to}" /> <child link="${ee_prefix}left_finger" />
+      <origin xyz="0 -0.006 0.015" rpy="0 0 0" /> <axis xyz="0 -1 0" />
       <limit effort="333" lower="0.0" upper="1.5708" velocity="10.0" />
       <mimic joint="${ee_prefix}finger_joint1" />

File: urdf/robot/openarm_robot.xacro (robot description, xacro)
@@ -18,5 +18,4 @@
             xyz:='0 0 0'
             rpy:='0 0 0'
-            hand:='false'
             ee_type:=''
             ros2_control:=false
@@ -46,5 +45,5 @@
     <xacro:include filename="$(find openarm_description)/urdf/body/openarm_body.xacro" />
     <xacro:include filename="$(find openarm_description)/urdf/ee/ee_dispatcher.xacro" />
-    <xacro:include filename="$(find openarm_description)/urdf/ee/openarm_hand_macro.xacro" />
+    <xacro:include filename="$(find openarm_description)/urdf/ee/openarm_ee_macro.xacro" />
     <xacro:include filename="$(find openarm_description)/urdf/ros2_control/openarm.ros2_control.xacro" />
     <xacro:include filename="$(find openarm_description)/urdf/ros2_control/openarm.bimanual.ros2_control.xacro" />
@@ -91,4 +90,20 @@
         kinematics_link="${kinematics_link}"
         kinematics_offset="${kinematics_offset}" />
+        <xacro:openarm_ee
+            connected_to="openarm_left_link7"
+            arm_type="${arm_type}"
+            arm_prefix="left_"
+            ee_type="${ee_type}"
+            ee_kinematics_link="${ee_kinematics_link}"
+            ee_inertials="${ee_inertials}"
+        />
+        <xacro:openarm_ee
+            connected_to="openarm_right_link7"
+            arm_type="${arm_type}"
+            arm_prefix="right_"
+            ee_type="${ee_type}"
+            ee_kinematics_link="${ee_kinematics_link}"
+            ee_inertials="${ee_inertials}"
+        />
         <!-- ros2_control hardware interfaces for bimanual setup -->
         <xacro:if value="${ros2_control}">
@@ -102,61 +117,38 @@
             left_arm_prefix="${left_arm_prefix}"
             right_arm_prefix="${right_arm_prefix}"
-            hand="${hand}"/>
-        </xacro:if>
-        <xacro:if value="${hand}">
-            <xacro:openarm_ee
-                connected_to="openarm_left_link7"
-                arm_type="${arm_type}"
-                arm_prefix="left_"
-                ee_type="${ee_type}"
-                ee_kinematics_link="${ee_kinematics_link}"
-                ee_inertials="${ee_inertials}"
-            />
-            <xacro:openarm_ee
-                connected_to="openarm_right_link7"
-                arm_type="${arm_type}"
-                arm_prefix="right_"
-                ee_type="${ee_type}"
-                ee_kinematics_link="${ee_kinematics_link}"
-                ee_inertials="${ee_inertials}"
-            />
+            hand="true"/>
         </xacro:if>
     </xacro:if>
     <xacro:if value="${not bimanual}">
         <xacro:openarm_arm
-        arm_type="${arm_type}"
-        arm_prefix="${arm_prefix_modified}"
-        no_prefix="${no_prefix}"
-        xyz="${xyz}"
-        rpy="${rpy}"
-        joint_limits="${joint_limits}"
-        kinematics="${kinematics}"
-        kinematics_link="${kinematics_link}"
-        inertials="${inertials}"
-        connected_to=""
+            arm_type="${arm_type}"
+            arm_prefix="${arm_prefix_modified}"
+            no_prefix="${no_prefix}"
+            xyz="${xyz}"
+            rpy="${rpy}"
+            joint_limits="${joint_limits}"
+            kinematics="${kinematics}"
+            kinematics_link="${kinematics_link}"
+            inertials="${inertials}"
+            connected_to=""
+        />
+        <xacro:openarm_ee
+            connected_to="openarm_${arm_prefix_modified}link7" arm_type="${arm_type}"
+            arm_prefix="${arm_prefix_modified}"
+            ee_type="${ee_type}"
+            ee_kinematics_link="${ee_kinematics_link}"
+            ee_inertials="${ee_inertials}"
         />
         <xacro:if value="${ros2_control}">
-        <xacro:openarm_arm_ros2_control
-            arm_type="${arm_type}"
-            control_gains="${control_gains}"
-            arm_prefix="${arm_prefix_modified}"
-            can_interface="${can_interface}"
-            use_fake_hardware="${use_fake_hardware}"
-            fake_sensor_commands="${fake_sensor_commands}"
-            hand="${hand}"
-            bimanual="false"
-            can_fd="${can_fd}"/>
-        </xacro:if>
-        <xacro:if value="${hand}">
-            <xacro:openarm_ee
-                connected_to="openarm_link7"
+            <xacro:openarm_arm_ros2_control
                 arm_type="${arm_type}"
+                control_gains="${control_gains}"
                 arm_prefix="${arm_prefix_modified}"
-                ee_type="${ee_type}"
-                ee_kinematics_link="${ee_kinematics_link}"
-                ee_inertials="${ee_inertials}"
-            />
-        </xacro:if>
-        </xacro:if>
+                can_interface="${can_interface}"
+                use_fake_hardware="${use_fake_hardware}"
+                fake_sensor_commands="${fake_sensor_commands}"
+                hand="true"
+                can_fd="${can_fd}"/> </xacro:if>
+    </xacro:if>
   </xacro:macro>
 </robot>

File: urdf/robot/v10/v10.urdf.xacro (robot description, xacro)
@@ -3,11 +3,7 @@
   <xacro:include filename="$(find openarm_description)/urdf/robot/openarm_robot.xacro"/>
   <xacro:arg name="arm_type" default="v10" />
+  <xacro:property name="auto_ee_type" value="${'parallel_link' if '$(arg arm_type)' == 'v10' else 'pinch_gripper'}" />
   <xacro:arg name="body_type" default="v10" />
-  <xacro:arg name="ee_type" default="parallel_gripper" />
   <xacro:arg name="no_prefix" default="false"/>
-  <xacro:arg name="hand" default="true" />
-  <xacro:if value="$(eval ee_type == 'none')">
-    <xacro:property name="hand" value="false"/>
-  </xacro:if>
   <xacro:arg name="parent" default="world" />
   <xacro:arg name="xyz" default="0 0 0" />
@@ -28,20 +24,16 @@
   <xacro:arg name="can_fd" default="true" />
   <xacro:openarm_robot
-  arm_type="v10"
-  body_type="v10"
-  joint_limits="${xacro.load_yaml('$(find openarm_description)/config/arm/v10/joint_limits.yaml')}"
-  control_gains="${xacro.load_yaml('$(find openarm_description)/config/arm/v10/control_gains.yaml')}"
-  inertials="${xacro.load_yaml('$(find openarm_description)/config/arm/v10/inertials.yaml')}"
-  kinematics="${xacro.load_yaml('$(find openarm_description)/config/arm/v10/kinematics.yaml')}"
-  kinematics_link="${xacro.load_yaml('$(find openarm_description)/config/arm/v10/kinematics_link.yaml')}"
-  kinematics_offset="${xacro.load_yaml('$(find openarm_description)/config/arm/v10/kinematics_offset.yaml')}"
-  body_inertials="${xacro.load_yaml('$(find openarm_description)/config/body/v10/inertials.yaml')}"
-  body_kinematics="${xacro.load_yaml('$(find openarm_description)/config/body/v10/kinematics.yaml')}"
-  body_kinematics_link="${xacro.load_yaml('$(find openarm_description)/config/body/v10/kinematics.yaml')}"
-  ee_kinematics_link="${xacro.load_yaml('$(find openarm_description)/config/hand/parallel_link/kinematics_link.yaml')}"
-  ee_inertials="${xacro.load_yaml('$(find openarm_description)/config/hand/parallel_link/inertials.yaml')}"
-  hand="$(arg hand)"
-  ee_type="$(arg ee_type)"
-  ros2_control="$(arg ros2_control)"
+  arm_type="$(arg arm_type)" body_type="$(arg body_type)" joint_limits="${xacro.load_yaml('$(find openarm_description)/config/arm/$(arg arm_type)/joint_limits.yaml')}"
+  control_gains="${xacro.load_yaml('$(find openarm_description)/config/arm/$(arg arm_type)/control_gains.yaml')}"
+  inertials="${xacro.load_yaml('$(find openarm_description)/config/arm/$(arg arm_type)/inertials.yaml')}"
+  kinematics="${xacro.load_yaml('$(find openarm_description)/config/arm/$(arg arm_type)/kinematics.yaml')}"
+  kinematics_link="${xacro.load_yaml('$(find openarm_description)/config/arm/$(arg arm_type)/kinematics_link.yaml')}"
+  kinematics_offset="${xacro.load_yaml('$(find openarm_description)/config/arm/$(arg arm_type)/kinematics_offset.yaml')}"
+  body_inertials="${xacro.load_yaml('$(find openarm_description)/config/body/$(arg body_type)/inertials.yaml')}"
+  body_kinematics="${xacro.load_yaml('$(find openarm_description)/config/body/$(arg body_type)/kinematics.yaml')}"
+  body_kinematics_link="${xacro.load_yaml('$(find openarm_description)/config/body/$(arg body_type)/kinematics.yaml')}"
+  ee_kinematics_link="${xacro.load_yaml('$(find openarm_description)/config/ee/' + auto_ee_type + '/kinematics_link.yaml')}"
+  ee_inertials="${xacro.load_yaml('$(find openarm_description)/config/ee/' + auto_ee_type + '/inertials.yaml')}"
+  ee_type="${auto_ee_type}" ros2_control="$(arg ros2_control)"
   can_interface="$(arg can_interface)"
   left_can_interface="$(arg left_can_interface)"

File: urdf/robot/v20/v20.urdf.xacro (robot description, xacro)
@@ -4,10 +4,6 @@
   <xacro:arg name="arm_type" default="v20" />
   <xacro:arg name="body_type" default="v20" />
-  <xacro:arg name="ee_type" default="pinch_gripper" />
+  <xacro:property name="auto_ee_type" value="${'parallel_link' if '$(arg arm_type)' == 'v10' else 'pinch_gripper'}" />
   <xacro:arg name="no_prefix" default="false"/>
-  <xacro:arg name="hand" default="true" />
-  <xacro:if value="$(eval ee_type == 'none')">
-    <xacro:property name="hand" value="false"/>
-  </xacro:if>
   <xacro:arg name="parent" default="world" />
   <xacro:arg name="xyz" default="0 0 0" />
@@ -28,19 +24,18 @@
   <xacro:arg name="can_fd" default="true" />
   <xacro:openarm_robot
-  arm_type="v20"
-  body_type="v20"
-  joint_limits="${xacro.load_yaml('$(find openarm_description)/config/arm/v20/joint_limits.yaml')}"
-  control_gains="${xacro.load_yaml('$(find openarm_description)/config/arm/v20/control_gains.yaml')}"
-  inertials="${xacro.load_yaml('$(find openarm_description)/config/arm/v20/inertials.yaml')}"
-  kinematics="${xacro.load_yaml('$(find openarm_description)/config/arm/v20/kinematics.yaml')}"
-  kinematics_link="${xacro.load_yaml('$(find openarm_description)/config/arm/v20/kinematics_link.yaml')}"
-  kinematics_offset="${xacro.load_yaml('$(find openarm_description)/config/arm/v20/kinematics_offset.yaml')}"
-  body_inertials="${xacro.load_yaml('$(find openarm_description)/config/body/v20/inertials.yaml')}"
-  body_kinematics="${xacro.load_yaml('$(find openarm_description)/config/body/v20/kinematics.yaml')}"
-  body_kinematics_link="${xacro.load_yaml('$(find openarm_description)/config/body/v20/kinematics_link.yaml')}"
-  ee_kinematics_link="${xacro.load_yaml('$(find openarm_description)/config/hand/pinch_gripper/kinematics_link.yaml')}"
-  ee_inertials="${xacro.load_yaml('$(find openarm_description)/config/hand/pinch_gripper/inertials.yaml')}"
-  hand="$(arg hand)"
-  ee_type="$(arg ee_type)"
+  arm_type="$(arg arm_type)"
+  body_type="$(arg body_type)"
+  joint_limits="${xacro.load_yaml('$(find openarm_description)/config/arm/$(arg arm_type)/joint_limits.yaml')}"
+  control_gains="${xacro.load_yaml('$(find openarm_description)/config/arm/$(arg arm_type)/control_gains.yaml')}"
+  inertials="${xacro.load_yaml('$(find openarm_description)/config/arm/$(arg arm_type)/inertials.yaml')}"
+  kinematics="${xacro.load_yaml('$(find openarm_description)/config/arm/$(arg arm_type)/kinematics.yaml')}"
+  kinematics_link="${xacro.load_yaml('$(find openarm_description)/config/arm/$(arg arm_type)/kinematics_link.yaml')}"
+  kinematics_offset="${xacro.load_yaml('$(find openarm_description)/config/arm/$(arg arm_type)/kinematics_offset.yaml')}"
+  body_inertials="${xacro.load_yaml('$(find openarm_description)/config/body/$(arg body_type)/inertials.yaml')}"
+  body_kinematics="${xacro.load_yaml('$(find openarm_description)/config/body/$(arg body_type)/kinematics.yaml')}"
+  body_kinematics_link="${xacro.load_yaml('$(find openarm_description)/config/body/$(arg body_type)/kinematics_link.yaml')}"
+  ee_kinematics_link="${xacro.load_yaml('$(find openarm_description)/config/ee/' + auto_ee_type + '/kinematics_link.yaml')}"
+  ee_inertials="${xacro.load_yaml('$(find openarm_description)/config/ee/' + auto_ee_type + '/inertials.yaml')}"
+  ee_type="${auto_ee_type}"
   ros2_control="$(arg ros2_control)"
   can_interface="$(arg can_interface)"
