Commit message: update docs and sync gripper configuration

File: assets/end_effector/pinch_gripper/urdf/pinch_gripper_standalone.urdf.xacro (robot description, xacro)
@@ -13,5 +13,4 @@
   <xacro:arg name="reflect_y" default="1" />
   <xacro:arg name="reflect_z" default="1" />
-  <xacro:arg name="swap_fingers" default="false" />
   <xacro:arg name="emit_grasp_frame" default="false" />
   <xacro:property name="reflect_x_value" value="${float('$(arg reflect_x)')}" lazy_eval="false" />
@@ -46,5 +45,4 @@
     reflect_include_reference_points="${list(ee_reference_points.keys())}"
     limit_override_joints="${dict()}"
-    swap_fingers="$(arg swap_fingers)"
     emit_grasp_frame="$(arg emit_grasp_frame)" />
 </robot>

File: assets/robot/openarm_v2.0/urdf/openarm_v20.urdf.xacro (robot description, xacro)
@@ -17,4 +17,7 @@
   <xacro:property name="gains_file" value="${config_root}/arm/control/control_gains.yaml" />
   <xacro:property name="gains_dict" value="${xacro.load_yaml(gains_file)}" />
+  <xacro:property name="pinch_mimics_file" value="$(find openarm_description)/assets/end_effector/pinch_gripper/config/joint/joint_mimics.yaml" />
+  <xacro:property name="pinch_mimics_dict" value="${xacro.load_yaml(pinch_mimics_file)}" />
+  <xacro:property name="pinch_finger_mimic_multiplier" value="${pinch_mimics_dict['joint2']['multiplier'] if 'joint2' in pinch_mimics_dict else 1.0}" />
   <xacro:openarm_bimanual_ros2_control
     arm_type="v20"
@@ -23,4 +26,6 @@
     ee_type="pinch_gripper"
     left_arm_prefix="left_"
-    right_arm_prefix="right_" />
+    right_arm_prefix="right_"
+    left_finger_mimic_multiplier="${pinch_finger_mimic_multiplier}"
+    right_finger_mimic_multiplier="${pinch_finger_mimic_multiplier}" />
 </robot>

File: assets/robot/openarm_v2.0/urdf/ros2_control/openarm.bimanual.ros2_control.xacro (robot description, xacro)
@@ -11,4 +11,6 @@
              left_arm_prefix:=^|left_
              right_arm_prefix:=^|right_
+             left_finger_mimic_multiplier:=^|1.0
+             right_finger_mimic_multiplier:=^|1.0
              can_fd:=^|true">
     <ros2_control name="openarm_left_hardware_interface" type="system">
@@ -68,5 +70,5 @@
       <joint name="openarm_${left_arm_prefix}finger_joint2">
         <param name="mimic">openarm_${left_arm_prefix}finger_joint1</param>
-        <param name="multiplier">-1.0</param>
+        <param name="multiplier">${left_finger_mimic_multiplier}</param>
         <command_interface name="position"/>
         <state_interface name="position">
@@ -114,5 +116,5 @@
       <joint name="openarm_${right_arm_prefix}finger_joint2">
         <param name="mimic">openarm_${right_arm_prefix}finger_joint1</param>
-        <param name="multiplier">-1.0</param>
+        <param name="multiplier">${right_finger_mimic_multiplier}</param>
         <command_interface name="position"/>
         <state_interface name="position">

File: assets/robot/openarm_v2.0/urdf/utils/openarm_v20_ee.xacro (robot description, xacro)
@@ -4,5 +4,5 @@
   <!-- Current EE implementation targets the two-finger gripper topology. -->
   <xacro:macro name="openarm_v20_ee"
-    params="prefix connected_to mount_origin:=none topology joint_origins joint_axes joint_limits joint_mimics inertials visuals collisions reflect_x:=1 reflect_y:=1 reflect_z:=1 component_reflects:=false reflect_include_links:=^ reflect_include_joints:=^ reflect_include_reference_points:=^ limit_override_joints:=^ swap_fingers:=false ee_reference_points:=^ emit_grasp_frame:=false grasp_reference_point:=grasp_frame skip_mount_joint:=false base_frame_shift:=none">
+    params="prefix connected_to mount_origin:=none topology joint_origins joint_axes joint_limits joint_mimics inertials visuals collisions reflect_x:=1 reflect_y:=1 reflect_z:=1 component_reflects:=false reflect_include_links:=^ reflect_include_joints:=^ reflect_include_reference_points:=^ limit_override_joints:=^ ee_reference_points:=^ emit_grasp_frame:=false grasp_reference_point:=grasp_frame skip_mount_joint:=false base_frame_shift:=none">
     <xacro:property name="base_link_name" value="${topology['links'][0]}" />
     <xacro:property name="base_link_full_name" value="${prefix}ee_${base_link_name}" />
@@ -11,5 +11,5 @@
     <xacro:property name="use_base_frame_shift" value="${base_frame_shift != 'none'}" lazy_eval="false" />
     <xacro:property name="base_link_reflects" value="${component_reflects and base_link_name in reflect_include_links}" lazy_eval="false" />
-    <!-- Keep joint/link numbering semantic: finger1 is inner, finger2 is outter. -->
+    <!-- Finger numbering stays semantic; handedness is handled by reflect_* and the joint config. -->
     <xacro:property name="finger1_source" value="link1" />
     <xacro:property name="finger2_source" value="link2" />
@@ -128,9 +128,9 @@
     <xacro:property
       name="finger1_limit_should_mirror"
-      value="${finger1_joint_axis_reflect_sign &lt; 0}"
+      value="${finger1_joint_reflects}"
       lazy_eval="false" />
     <xacro:property
       name="finger2_limit_should_mirror"
-      value="${finger2_joint_axis_reflect_sign &lt; 0}"
+      value="${finger2_joint_reflects}"
       lazy_eval="false" />
     <xacro:property

File: assets/robot/openarm_v2.0/urdf/utils/openarm_v20_robot.xacro (robot description, xacro)
@@ -248,5 +248,4 @@
     <xacro:property name="reflect_include_reference_points" value="${reflect_include_cfg['reference_points'] if 'reference_points' in reflect_include_cfg else list(component_desc['reference_points'].keys())}" lazy_eval="false" />
     <xacro:property name="limit_override_joints" value="${component_cfg['limit_override_joints'] if 'limit_override_joints' in component_cfg else dict()}" lazy_eval="false" />
-    <xacro:property name="swap_fingers" value="${component_cfg['swap_fingers'] if 'swap_fingers' in component_cfg else False}" lazy_eval="false" />
     <xacro:property name="connection" value="${component_cfg['connection'] if 'connection' in component_cfg else dict()}" lazy_eval="false" />
     <xacro:property name="parent_component_name" value="${connection['attach_to'] if 'attach_to' in connection else none_value}" lazy_eval="false" />
@@ -360,5 +359,4 @@
                    reflect_include_reference_points=reflect_include_reference_points,
                    limit_override_joints=limit_override_joints,
-                   swap_fingers=swap_fingers,
                    resolved_connected_to=resolved_connected_to,
                    resolved_mount_origin=resolved_mount_origin,
@@ -438,5 +436,4 @@
         reflect_include_reference_points="${component_runtime['reflect_include_reference_points']}"
         limit_override_joints="${component_runtime['limit_override_joints']}"
-        swap_fingers="${component_runtime['swap_fingers']}"
         emit_grasp_frame="${emit_grasp_frame}"
         skip_mount_joint="${component_runtime['skip_mount_joint']}"
