Commit message: delete bug joint setting in ros2 controller

File: assets/robot/openarm_v2.0/urdf/ros2_control/openarm.bimanual.ros2_control.xacro (robot description, xacro)
@@ -68,5 +68,5 @@
       <xacro:configure_joint joint_name="openarm_${left_arm_prefix}joint7" initial_position="0.0"/>
       <xacro:configure_joint joint_name="openarm_${left_arm_prefix}finger_joint1" initial_position="0.0" />
-      <joint name="openarm_${left_arm_prefix}finger_joint2">
+      <!-- <joint name="openarm_${left_arm_prefix}finger_joint2">
         <param name="mimic">openarm_${left_arm_prefix}finger_joint1</param>
         <param name="multiplier">${left_finger_mimic_multiplier}</param>
@@ -75,5 +75,5 @@
           <param name="initial_value">0.0</param>
         </state_interface>
-      </joint>
+      </joint> -->
     </ros2_control>
     <ros2_control name="openarm_right_hardware_interface" type="system">
@@ -114,5 +114,5 @@
       <xacro:configure_joint joint_name="openarm_${right_arm_prefix}joint7" initial_position="0.0"/>
       <xacro:configure_joint joint_name="openarm_${right_arm_prefix}finger_joint1" initial_position="0.0" />
-      <joint name="openarm_${right_arm_prefix}finger_joint2">
+      <!-- <joint name="openarm_${right_arm_prefix}finger_joint2">
         <param name="mimic">openarm_${right_arm_prefix}finger_joint1</param>
         <param name="multiplier">${right_finger_mimic_multiplier}</param>
@@ -121,5 +121,5 @@
           <param name="initial_value">0.0</param>
         </state_interface>
-      </joint>
+      </joint> -->
     </ros2_control>
   </xacro:macro>
